File: frontend/basic 1w pa/basic-1W-pa.kicad_pcb (KiCad board)
At the start: 2 copper layers, 97 x 83 mm, 84 parts, among them CN1 EDGE, CN2 BREAKOUT, K1 IM23TS, P1 BNC, P2 CONN_01X02, P3 CONN_01X02, P4 CONN_01X02, P5 CONN_02X01, P6 +S12V, Q10 BS170, Q11 BS170, Q3 BS170, Q4 2N3906, Q5 BS170, Q6 2N3904, Q7 BS170, Q8 BS170, Q9 PZT2222A, T1 4:1, T2 8:1, T3 TRANSF, T4 TRANSF, T5 TRANSFO

Commit message: Version 1.7 updates
Parts:
- removed C1, C2: 0.1 uF, Capacitors_SMD:C_0805_HandSoldering
- removed CN2: BREAKOUT, Pin_Headers:Pin_Header_Straight_1x12
- removed D1: TVS DIODE, HERMESLITE:SOD323
- removed D3: 1N4003, Diodes_SMD:Diode-SMB_Handsoldering
- removed the MH at (173.0, 108.4)
- removed the MH at (184.8, 58.6)
- removed the MH at (184.8, 131.2)
- removed the MH at (105.8, 130.8)
- removed the MH at (105.8, 58.4)
- removed Q10, Q11: BS170, Housings_TO-92:TO-92-Free-inline-wide
- added C26: 2700pF, Capacitors_SMD:C_0805_HandSoldering, F.Cu at (153.8, 154.4)
- added C27: 4700pF, Capacitors_SMD:C_0805_HandSoldering, F.Cu at (184.2, 155.0)
- added C28: 33pF, Capacitors_SMD:C_0805_HandSoldering, F.Cu at (130.0, 115.8)
- added C29: 47pF, Capacitors_SMD:C_0805_HandSoldering, F.Cu at (160.6, 115.8)
- added C30: 82pF, Capacitors_SMD:C_0805_HandSoldering, F.Cu at (191.2, 115.4)
- added C31: 300pF, Capacitors_SMD:C_0805_HandSoldering, F.Cu at (127.8, 154.8)
- added C32: 270pF, Capacitors_SMD:C_0805_HandSoldering, F.Cu at (159.6, 154.4)
- added C33: 690pF, Capacitors_SMD:C_0805_HandSoldering, F.Cu at (190.2, 155.0)
- added C34: 182pF, Capacitors_SMD:C_0805_HandSoldering, F.Cu at (135.8, 116.0)
- added C35: 270pF, Capacitors_SMD:C_0805_HandSoldering, F.Cu at (166.8, 115.8)
- added C36: 390pF, Capacitors_SMD:C_0805_HandSoldering, F.Cu at (197.4, 115.4)
- added C37: 820pF, Capacitors_SMD:C_0805_HandSoldering, F.Cu at (135.2, 154.8)
- added C38: 1500pF, Capacitors_SMD:C_0805_HandSoldering, F.Cu at (167.4, 154.2)
- added C39: 2200pF, Capacitors_SMD:C_0805_HandSoldering, F.Cu at (195.8, 155.0)
- added K10: D3002, Sockets_DIP:DIP-10__300, F.Cu at (131.4, 135.6)
- added K11: D3002, Sockets_DIP:DIP-10__300, F.Cu at (163.0, 135.2)
- added K12: D3002, Sockets_DIP:DIP-10__300, F.Cu at (193.4, 135.6)
- added K2: D3002, Sockets_DIP:DIP-10__300, F.Cu at (148.0, 96.2)
- added K3: D3002, Sockets_DIP:DIP-10__300, F.Cu at (179.4, 96.6)
- added K4: D3002, Sockets_DIP:DIP-10__300, F.Cu at (116.0, 135.6)
- added K5: D3002, Sockets_DIP:DIP-10__300, F.Cu at (147.6, 135.4)
- added K6: D3002, Sockets_DIP:DIP-10__300, F.Cu at (178.4, 135.6)
- added K7: D3002, Sockets_DIP:DIP-10__300, F.Cu at (131.4, 96.4)
- added K8: D3002, Sockets_DIP:DIP-10__300, F.Cu at (162.8, 96.2)
- added K9: D3002, Sockets_DIP:DIP-10__300, F.Cu at (192.8, 96.4)
- added L11: 400nH, Choke_Toroid_ThroughHole:Choke_Toroid_6,5x13mm_Vertical, F.Cu at (138.0, 146.0)
- added L12: 676nH, Choke_Toroid_ThroughHole:Choke_Toroid_6,5x13mm_Vertical, F.Cu at (169.2, 145.6)
- added L13: 1.6uH, Choke_Toroid_ThroughHole:Choke_Toroid_6,5x13mm_Vertical, F.Cu at (199.8, 145.8)
- added L14: 1.083uH, Choke_Toroid_ThroughHole:Choke_Toroid_6,5x13mm_Vertical, F.Cu at (128.0, 118.4)
- added L15: 1.452uH, Choke_Toroid_ThroughHole:Choke_Toroid_6,5x13mm_Vertical, F.Cu at (157.2, 118.4)
- added L16: 2.028uH, Choke_Toroid_ThroughHole:Choke_Toroid_6,5x13mm_Vertical, F.Cu at (187.0, 118.4)
- added L17: 3.6uH, Choke_Toroid_ThroughHole:Choke_Toroid_6,5x13mm_Vertical, F.Cu at (124.4, 157.4)
- added L18: 7.396uH, Choke_Toroid_ThroughHole:Choke_Toroid_6,5x13mm_Vertical, F.Cu at (155.4, 157.4)
- added L19: 11.664uH, Choke_Toroid_ThroughHole:Choke_Toroid_6,5x13mm_Vertical, F.Cu at (186.2, 157.4)
- added L20: 192nH, Choke_Toroid_ThroughHole:Choke_Toroid_6,5x13mm_Vertical, F.Cu at (129.0, 125.0)
- added L21: 243nH, Choke_Toroid_ThroughHole:Choke_Toroid_6,5x13mm_Vertical, F.Cu at (158.6, 125.0)
- added L22: 432nH, Choke_Toroid_ThroughHole:Choke_Toroid_6,5x13mm_Vertical, F.Cu at (189.0, 124.8)
- added L23: 784nH, Choke_Toroid_ThroughHole:Choke_Toroid_6,5x13mm_Vertical, F.Cu at (126.4, 164.0)
- added L24: 1.296uH, Choke_Toroid_ThroughHole:Choke_Toroid_6,5x13mm_Vertical, F.Cu at (157.2, 163.8)
- added L25: 3.364uH, Choke_Toroid_ThroughHole:Choke_Toroid_6,5x13mm_Vertical, F.Cu at (187.8, 164.0)
- added L9: 108nH, Choke_Toroid_ThroughHole:Choke_Toroid_6,5x13mm_Vertical, F.Cu at (169.2, 106.6)
- added MH: VAL**, HERMESLITE:MH, F.Cu at (178.9, 67.9)
- added MH: VAL**, HERMESLITE:MH, F.Cu at (209.0, 54.0)
- added MH: VAL**, HERMESLITE:MH, F.Cu at (108.0, 54.0)
- added MH: VAL**, HERMESLITE:MH, F.Cu at (108.0, 167.0)
- added MH: VAL**, HERMESLITE:MH, F.Cu at (209.0, 167.0)
- added Q1: BS170, Housings_TO-92:TO-92-Free-inline-wide, F.Cu at (120.6, 64.2)
- added Q2: 2N3906, Transistors_SMD:sot23, F.Cu at (159.4, 61.6)
- added U1: ULN2003A, Sockets_DIP:DIP-16__300, F.Cu at (131.2, 75.2)
- C10, C12, C13, C8: value C -> 0.01uF
- C11: value C -> 220pF
- C14, C7: value C -> 47uF 16V; footprint Capacitors_SMD:C_0805_HandSoldering -> Discret:C1V8
- C16: value 47uF 16V -> 68pF; footprint Discret:C1V8 -> Capacitors_SMD:C_0805_HandSoldering
- C17, C19: value 0.01uF -> 100pF
- C18: value 0.01uF -> 150pF
- C20: value 0.1uF -> 550pF
- C21: value 0.01uF -> 1500pF
- C22: value 220pF -> 472pF
- C23: value 0.1uF -> 630pF
- C24: value 47uF 16V -> 690pF; footprint Discret:C1V8 -> Capacitors_SMD:C_0805_HandSoldering
- C25: value 0.1uF -> 1600pF
- C4: value 0.1uF -> 0.1 uF
- C5: value C -> 0.1 uF
- C6, C9: value C -> 0.1uF
- K1: value IM23TS -> D3002; footprint HERMESLITE:IM23TS -> Sockets_DIP:DIP-10__300
- L1: footprint Choke_Toroid_ThroughHole:Choke_Toroid_6,5x13mm_Vertical -> Choke_Axial_ThroughHole:Choke_Horizontal_RM10mm
- L10: value INDUCTOR -> 243nH; footprint Choke_Axial_ThroughHole:Choke_Horizontal_RM10mm -> Choke_Toroid_ThroughHole:Choke_Toroid_6,5x13mm_Vertical
- L2: value INDUCTOR -> 507nH
- L3: value INDUCTOR -> 675nH
- L4: value INDUCTOR -> 1.083uH
- L5: value INDUCTOR -> 1.936uH
- L6: value INDUCTOR -> 3.364uH
- L7: value INDUCTOR -> 5.184uH
- L8: value INDUCTOR -> 75nH
- P1: value BNC -> CONN_01X02; footprint HERMESLITE:BNCRA -> Pin_Headers:Pin_Header_Angled_1x02
- P2: value CONN_01X02 -> CONN_02X01
- P4: value CONN_01X02 -> CONN_01X07; footprint Pin_Headers:Pin_Header_Straight_1x02 -> Pin_Headers:Pin_Header_Straight_1x07
- P5: value CONN_02X01 -> DGND; footprint Pin_Headers:Pin_Header_Straight_2x01 -> Pin_Headers:Pin_Header_Straight_1x01
- P6: value +S12V -> CONN_01X03; footprint Pin_Headers:Pin_Header_Straight_1x02 -> Pin_Headers:Pin_Header_Straight_1x03
- Q3: value BS170 -> PZT2222A; footprint Housings_TO-92:TO-92-Free-inline-wide -> SMD_Packages:SOT-223
- Q4: value 2N3906 -> BS170; footprint Transistors_SMD:sot23 -> Housings_TO-92:TO-92-Free-inline-wide
- Q5: value BS170 -> 2N3904; footprint Housings_TO-92:TO-92-Free-inline-wide -> Transistors_SMD:sot23
- Q6: value 2N3904 -> BS170; footprint Transistors_SMD:sot23 -> Housings_TO-92:TO-92-Free-inline-wide
- Q9: value PZT2222A -> BS170; footprint SMD_Packages:SOT-223 -> Housings_TO-92:TO-92-Free-inline-wide
- R10: value 221 -> 2.21k
- R11: value 2.21 -> 68.1
- R12: value 221 -> 33.2
- R13: value 2.21 -> 221
- R14: value 68.1 -> 221
- R15: value 56.2 -> 2.21
- R16: value 475 -> 2.21
- R17: value 2.21k -> 22.1k
- R18: value 0 -> 221
- R3: value 4.99k -> 0
- R4: value 1k -> 4.99k
- R5: value 22.1 -> 1k
- R7: value 33.2 -> 475
- R8: value 22.1k -> 22.1
- R9: value 221 -> 56.2
- T1: value 4:1 -> TRANSFO; footprint HERMESLITE:TRANSF -> Socket_Strips:Socket_Strip_Straight_2x02
- T3: value TRANSF -> 4:1
- T5: value TRANSFO -> TRANSF; footprint Socket_Strips:Socket_Strip_Straight_2x02 -> HERMESLITE:TRANSF
- moved P2 114.5 mm to (105.8, 150.2), turned to 90 degrees
- moved C10 109.4 mm to (192.4, 56.4)
- moved C13 101.5 mm to (199.4, 75.2), turned to 270 degrees
- moved C19 89.2 mm to (123.6, 143.2)
- moved L1 88.6 mm to (206.8, 82.4), turned to 270 degrees
- moved C14 81.6 mm to (202.4, 60.0), turned to 180 degrees
- moved T5 80.2 mm to (200.8, 71.0)
- moved D2 79.2 mm to (176.0, 56.8), turned to 180 degrees
- moved C21 78.3 mm to (186.0, 143.8)
- moved C12 69.4 mm to (191.4, 83.4)
- moved R7 68.8 mm to (129.2, 58.2), turned to 180 degrees
- moved L7 65.7 mm to (172.0, 152.4)
- moved L10 64.0 mm to (200.6, 106.6), turned to 180 degrees
- moved C15 63.4 mm to (165.2, 67.0)
- moved R9 61.4 mm to (135.6, 58.2), turned to 180 degrees
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Connections:
- net Net-(CN1-PadA15) renamed +3V
- C10 pad 2: Net-(C10-Pad2) -> GND
- C13 pad 1: Net-(C10-Pad1) -> Net-(C13-Pad1)
- C14 pad 1: Net-(C11-Pad1) -> Net-(C13-Pad1)
- C15 pad 1: Net-(C15-Pad1) -> Net-(C12-Pad1)
- C16 pad 1: Net-(C15-Pad1) -> Net-(C16-Pad1)
- C16 pad 2: GND -> Net-(C16-Pad2)
- C17 pad 2: GND -> Net-(C17-Pad2)
- C18 pad 2: GND -> Net-(C18-Pad2)
- C19 pad 1: Net-(C18-Pad1) -> Net-(C19-Pad1)
- C19 pad 2: GND -> Net-(C19-Pad2)
- C20 pad 2: GND -> Net-(C20-Pad2)
- C22 pad 1: Net-(C22-Pad1) -> Net-(C16-Pad2)
- C22 pad 2: Net-(C22-Pad2) -> GND
- C23 pad 1: Net-(C23-Pad1) -> Net-(C17-Pad2)
- C24 pad 1: Net-(C24-Pad1) -> Net-(C18-Pad2)
- C25 pad 1: Net-(C24-Pad1) -> Net-(C19-Pad2)
- C3 pad 2: Net-(C3-Pad2) -> GND
- C4 pad 1: Net-(C3-Pad2) -> Net-(C4-Pad1)
- C4 pad 2: Net-(C4-Pad2) -> GND
- C5 pad 2: Net-(C5-Pad2) -> GND
- C6 pad 1: Net-(C6-Pad1) -> +12V
- C6 pad 2: Net-(C6-Pad2) -> GND
- C7 pad 1: Net-(C7-Pad1) -> +12V
- C8 pad 1: Net-(C5-Pad2) -> Net-(C8-Pad1)
- C8 pad 2: GND -> Net-(C8-Pad2)
- C9 pad 1: Net-(C6-Pad2) -> S12V
- CN1 pad A11: Net-(C24-Pad1) -> +12V
- CN1 pad A12: Net-(C24-Pad1) -> +12V
- CN1 pad B12: GPIO0 -> 160M
- CN1 pad B13: Net-(CN1-PadB13) -> 80/75M
- CN1 pad B14: Net-(CN1-PadB14) -> 60/40M
- CN1 pad B15: Net-(CN1-PadB15) -> 30/20M
- CN1 pad B16: Net-(CN1-PadB16) -> 17/15M
- CN1 pad B17: Net-(CN1-PadB17) -> 10/12M
- D2 pad 1: GND -> Net-(D2-Pad1)
- D2 pad 2: GPIO0 -> Net-(C12-Pad1)
- K1 pad 1: GPIO0 -> +12V
- K1 pad 2: Net-(C11-Pad1) -> Net-(K1-Pad2)
- K1 pad 3: Net-(K1-Pad3) -> ANT
- K1 pad 4: Net-(C6-Pad2) -> Net-(K1-Pad4)
- K1 pad 5: Net-(C12-Pad1) -> (no net)
- K1 pad 6: Net-(K1-Pad6) -> (no net)
- K1 pad 7: Net-(C7-Pad1) -> Net-(K1-Pad4)
- K1 pad 8: GND -> ANT
- L1 pad 1: Net-(C7-Pad1) -> Net-(C13-Pad1)
- L1 pad 2: Net-(C5-Pad1) -> +12V
- L10 pad 1: Net-(C15-Pad1) -> Net-(C18-Pad2)
- L10 pad 2: Net-(C24-Pad1) -> GND
- L2 pad 1: Net-(C5-Pad2) -> Net-(K1-Pad2)
- L2 pad 2: Net-(C6-Pad1) -> Net-(C16-Pad1)
- L3 pad 1: Net-(C6-Pad2) -> Net-(K2-Pad2)
- L3 pad 2: GND -> Net-(C17-Pad1)
- L4 pad 1: Net-(C5-Pad2) -> Net-(K3-Pad2)
- L4 pad 2: GND -> Net-(C18-Pad1)
- L5 pad 1: Net-(C10-Pad2) -> Net-(K4-Pad2)
- L5 pad 2: Net-(C12-Pad1) -> Net-(C19-Pad1)
- L6 pad 1: Net-(C11-Pad2) -> Net-(K5-Pad2)
- L6 pad 2: Net-(C10-Pad1) -> Net-(C20-Pad1)
- L7 pad 1: Net-(C11-Pad1) -> Net-(K6-Pad2)
- L7 pad 2: GND -> Net-(C21-Pad1)
- L8 pad 1: Net-(C10-Pad1) -> Net-(C16-Pad2)
- P1 pad 1: Net-(C3-Pad1) -> Net-(P1-Pad1)
- P1 pad 2: Net-(D1-Pad2) -> Net-(P1-Pad2)
- P2 pad 2: GND -> Net-(P1-Pad1)
- P3 pad 1: GND -> Net-(CN1-PadB9)
- P3 pad 2: GND -> Net-(CN1-PadB8)
- P4 pad 1: Net-(CN1-PadB9) -> Net-(K1-Pad10)
- P4 pad 2: Net-(CN1-PadB8) -> Net-(K2-Pad10)
- P5 pad 1: GND -> Net-(CN1-PadA17)
- P6 pad 1: GND -> PTT#
- P6 pad 2: Net-(C20-Pad1) -> Net-(P6-Pad2)
- Q3 pad 1: Net-(K1-Pad3) -> Net-(C8-Pad1)
- Q3 pad 2: Net-(C23-Pad1) -> Net-(Q3-Pad2)
- Q3 pad 3: Net-(Q3-Pad3) -> Net-(C11-Pad2)
- Q4 pad 1: Net-(C24-Pad1) -> Net-(C10-Pad1)
- Q4 pad 2: Net-(Q4-Pad2) -> Net-(D2-Pad1)
- Q4 pad 3: Net-(C20-Pad1) -> Net-(P6-Pad2)
- Q5 pad 1: Net-(Q5-Pad1) -> GND
- Q5 pad 2: Net-(D3-Pad1) -> Net-(P6-Pad2)
- Q6 pad 1: GND -> Net-(Q6-Pad1)
- Q6 pad 2: Net-(Q5-Pad3) -> Net-(Q6-Pad2)
- Q7 pad 1: Net-(Q10-Pad1) -> Net-(Q7-Pad1)
- Q7 pad 2: Net-(Q10-Pad2) -> Net-(Q7-Pad2)
- Q7 pad 3: Net-(Q10-Pad3) -> Net-(Q7-Pad3)
- Q8 pad 1: Net-(Q11-Pad1) -> Net-(Q6-Pad1)
- Q8 pad 2: Net-(Q11-Pad2) -> Net-(Q6-Pad2)
- Q8 pad 3: Net-(Q11-Pad3) -> Net-(Q6-Pad3)
- Q9 pad 1: Net-(C21-Pad1) -> Net-(Q7-Pad1)
- Q9 pad 2: Net-(Q9-Pad2) -> Net-(Q7-Pad2)
- Q9 pad 3: Net-(C22-Pad2) -> Net-(Q7-Pad3)
- R1 pad 1: Net-(C23-Pad1) -> Net-(C3-Pad1)
- R10 pad 1: Net-(Q11-Pad2) -> Net-(D2-Pad1)
- R10 pad 2: Net-(C18-Pad1) -> Net-(C10-Pad1)
- R11 pad 1: Net-(Q11-Pad3) -> Net-(C11-Pad1)
- R12 pad 1: Net-(C18-Pad1) -> Net-(P6-Pad2)
- R12 pad 2: Net-(Q10-Pad2) -> GND
- R13 pad 1: Net-(Q10-Pad3) -> Net-(Q6-Pad2)
- R13 pad 2: GND -> Net-(C12-Pad1)
- R14 pad 1: Net-(C22-Pad1) -> Net-(C12-Pad1)
- R14 pad 2: GND -> Net-(Q7-Pad2)
- R15 pad 1: Net-(C22-Pad2) -> Net-(Q6-Pad3)
- R16 pad 1: Net-(C21-Pad1) -> Net-(Q7-Pad3)
- R17 pad 1: Net-(Q9-Pad2) -> Net-(Q5-Pad3)
- R17 pad 2: Net-(C21-Pad1) -> GND
- R18 pad 1: Net-(C1-Pad1) -> Net-(Q5-Pad3)
- R18 pad 2: Net-(FB1-Pad2) -> Net-(C12-Pad1)
- R2 pad 1: Net-(C23-Pad1) -> Net-(C3-Pad1)
- R3 pad 1: PTT# -> Net-(C5-Pad1)
- R3 pad 2: Net-(Q4-Pad2) -> Net-(FB1-Pad2)
- R4 pad 1: Net-(C24-Pad1) -> PTT#
- R4 pad 2: Net-(Q4-Pad2) -> Net-(Q2-Pad2)
- R5 pad 1: Net-(Q5-Pad1) -> +12V
- R5 pad 2: Net-(C20-Pad1) -> Net-(Q2-Pad2)
- R6 pad 1: Net-(D3-Pad1) -> Net-(Q3-Pad2)
- R6 pad 2: Net-(Q5-Pad1) -> Net-(C8-Pad1)
- R7 pad 1: Net-(Q5-Pad3) -> Net-(C8-Pad1)
- R8 pad 1: Net-(Q6-Pad3) -> Net-(C10-Pad1)
- R8 pad 2: GND -> S12V
- R9 pad 1: Net-(Q6-Pad3) -> Net-(C11-Pad2)
- R9 pad 2: Net-(C18-Pad1) -> GND
- T1 pad 1: Net-(C21-Pad2) -> Net-(P1-Pad2)
- T1 pad 2: GND -> Net-(P1-Pad1)
- T1 pad 3: Net-(C1-Pad1) -> GND
- T1 pad 4: Net-(CN1-PadB5) -> ANT
- T2 pad 1: Net-(Q3-Pad3) -> Net-(Q1-Pad3)
- T2 pad 3: Net-(C2-Pad1) -> Net-(C4-Pad1)
- T2 pad 6: Net-(C2-Pad1) -> Net-(C4-Pad1)
- T3 pad 1: Net-(C17-Pad1) -> Net-(C8-Pad2)
- T3 pad 2: Net-(Q9-Pad2) -> GND
- T3 pad 3: Net-(C18-Pad1) -> Net-(C5-Pad1)
- T3 pad 4: Net-(Q11-Pad2) -> Net-(CN1-PadB5)
- T3 pad 5: Net-(Q10-Pad2) -> Net-(CN1-PadB6)
- T3 pad 6: Net-(C18-Pad1) -> Net-(C5-Pad1)
- T4 pad 1: Net-(K1-Pad3) -> Net-(C10-Pad1)
- T4 pad 2: GND -> Net-(Q3-Pad2)
- T4 pad 3: Net-(C15-Pad1) -> Net-(C12-Pad1)
- T4 pad 4: Net-(Q10-Pad1) -> Net-(Q6-Pad2)
- T4 pad 5: Net-(Q11-Pad1) -> Net-(Q7-Pad2)
- T4 pad 6: Net-(C15-Pad1) -> Net-(C12-Pad1)
- T5 pad 1: Net-(C4-Pad2) -> RX/TX
- T5 pad 2: Net-(D1-Pad2) -> GND
- T5 pad 3: GND -> Net-(C13-Pad1)
- T5 pad 4: Net-(K1-Pad6) -> Net-(Q7-Pad1)
Routing:
- net GND: track 0.00 -> 803.8 mm, vias 0 -> 6
- net +12V: track 0.00 -> 330.1 mm, vias 0 -> 3
- net Net-(K3-Pad10): track 0.00 -> 197.9 mm, vias 0 -> 6
- net Net-(K12-Pad10): track 0.00 -> 194.0 mm, vias 0 -> 3
- net RX/TX: track 0.00 -> 180.1 mm, vias 0 -> 6
- net Net-(K10-Pad3): track 0.00 -> 138.1 mm, vias 0 -> 4
- net Net-(K11-Pad10): track 0.00 -> 135.5 mm, vias 0 -> 5
- net Net-(K10-Pad10): track 0.00 -> 119.0 mm, vias 0 -> 3
- net Net-(K2-Pad10): track 0.00 -> 110.1 mm, vias 0 -> 3
- net Net-(K3-Pad4): track 0.00 -> 109.5 mm, vias 0 -> 2
- net Net-(C12-Pad1): track 0.00 -> 91.8 mm, vias 0 -> 2
- net Net-(Q6-Pad2): track 0.00 -> 74.7 mm, vias 0 -> 1
- net Net-(P6-Pad2): track 0.00 -> 73.2 mm, vias 0 -> 8
- net Net-(K1-Pad10): track 0.00 -> 69.8 mm
- net Net-(C10-Pad1): track 0.00 -> 66.9 mm
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Other:
- board size 97 x 83 mm -> 115 x 126.8 mm
