File: frontend/basic 1w pa/basic-1W-pa.sch (KiCad schematic (older format))
At the start: 79 parts, among them CN1 EDGE, CN2 BREAKOUT, K1 IM23TS, P1 BNC, P2 CONN_01X02, P3 CONN_01X02, P4 CONN_01X02, P5 CONN_02X01, P6 +S12V, Q10 BS170, Q11 BS170, Q3 BS170, Q4 2N3906, Q5 BS170, Q6 2N3904, Q7 BS170, Q8 BS170, Q9 PZT2222A, T1 4:1, T2 8:1, T3 TRANSF, T4 TRANSF, T5 TRANSFO

Commit message: Version 1.7 updates
Parts:
- removed C10, C11, C12, C13, C14, C5, C6, C7, C8, C9: C, Capacitors_SMD:C_0805_HandSoldering, symbol C
- removed C3, C4: 0.1uF, Capacitors_SMD:C_0805_HandSoldering, symbol C
- removed CN2: BREAKOUT, Pin_Headers:Pin_Header_Straight_1x12, symbol BREAKOUT
- removed D1: TVS DIODE, HERMESLITE:SOD323, symbol DIODESCH2
- removed D2: 1N4003, Diodes_SMD:Diode-SMB_Handsoldering, symbol DIODE
- removed K1: IM23TS, HERMESLITE:IM23TS, symbol IM23TS
- removed L1, L2, L3, L4, L5, L6, L7, L8: INDUCTOR, Choke_Toroid_ThroughHole:Choke_Toroid_6,5x13mm_Vertical, symbol INDUCTOR
- removed P1: BNC, HERMESLITE:BNCRA, symbol BNC
- removed P2, P3: CONN_01X02, Pin_Headers:Pin_Header_Straight_1x02, symbol CONN_01X02
- removed P6: +S12V, Pin_Headers:Pin_Header_Straight_1x02, symbol CONN_01X02
- added P1: CONN_01X02, Pin_Headers:Pin_Header_Angled_1x02, symbol CONN_01X02
- added P5: DGND, Pin_Headers:Pin_Header_Straight_1x01, symbol CONN_01X01
- added P6: CONN_01X03, Pin_Headers:Pin_Header_Straight_1x03, symbol CONN_01X03
- P2: renamed from P5; footprint Pin_Headers:Pin_Header_Straight_2x01 -> Pin_Headers:Pin_Header_Straight_1x02
- renumbered C17 to C10, C22 to C11, C18 to C12, C15 to C13, C16 to C14, C19 to C15, C23 to C3, C2 to C4, C1 to C5, C25 to C6, C24 to C7, C21 to C8, C20 to C9, D3 to D2, L10 to L1, P4 to P3, Q3 to Q1, Q4 to Q2, Q9 to Q3, Q5 to Q4, Q6 to Q5, Q8 to Q6, Q11 to Q8, Q10 to Q9, R6 to R10, R14 to R11, R7 to R12, R10 to R13, R12 to R14, R11 to R15, R13 to R16, R8 to R17, R9 to R18, R18 to R3, R3 to R4, R4 to R5, R17 to R6, R16 to R7, R5 to R8, R15 to R9, T5 to T1, T1 to T3, T3 to T4, T4 to T5
Connections:
- net GND: now also P6.3 (P3)
- net PTT#: now also P6.1 (P1)
- net +12V: now reaches C6.1, C7.1, CN1.A11 (12V), CN1.A12 (12V), L1.2, Q2.1 (E), R5.1
- net +3V: now reaches CN1.A15 (3V), CN1.A16 (3V)
- net at CN1.A17 (DGND), CN1.A18 (DGND): now also P5.1 (P1)
- net 80/75M: now reaches CN1.B13 (GPIO1)
- net 60/40M: now reaches CN1.B14 (GPIO2)
- net 30/20M: now reaches CN1.B15 (SEN)
- net 17/15M: now reaches CN1.B16 (SDI)
- net 10/12M: now reaches CN1.B17 (SDO)
- net at C10.1, T4.1 (S1): now also Q4.1 (D), R10.2, R8.1
- net RX/TX: now reaches Q1.1 (D), T5.1 (S1)
- net at Q4.3 (S), Q5.2 (B), R12.1: now also P6.2 (P2)
- net S12V: now reaches C9.1, Q2.3 (C), R8.2
- net at P2.2 (P2), T1.2 (AB): now also P1.1 (P1)
- net at T1.1 (AA): now also P1.2 (P2)
- net ANT: now reaches T1.4 (SB)
- net GPIO0 renamed 160M
Other:
- note added: "BN-43-2402\n 6T 2x3T #30"
- note added: "S12V"
- note removed: "(Band Specific Values)"
- note removed: "BN-43-2402 L\nBN-61-2402 H\n 6T 2x3T #30"
- note removed: "Filter\nControl"
- note removed: "Note: When not using SPI, 3 GPIO signals are available. \nGPIO0 is band select.\nIf SPI is used, GPIO2 becomes SEN1 (Transmit Strobe - Alex Protocol)\nSEN should be called SEN0 (Receive Strobe - Alex Protocol)\n"
- note removed: "Omitted for\nlower freq's"
- moved on the sheet: P2
