File: frontend/basic 1w pa/basic-1W-pa - Copy.sch (KiCad schematic (older format))
At the start: 54 parts, among them CN1 EDGE, P1 CONN_01X02, P2 CONN_02X01, P3 CONN_01X02, P5 DGND, P6 CONN_01X03, Q1 BS170, Q2 2N3906, Q3 PZT2222A, Q4 BS170, Q5 2N3904, Q6 BS170, Q7 BS170, Q8 BS170, Q9 BS170, T1 TRANSFO, T2 8:1, T3 4:1, T4 TRANSF, T5 TRANSF

Commit message: 10W amp initial commit
Parts:
- removed P1: CONN_01X02, Pin_Headers:Pin_Header_Angled_1x02, symbol CONN_01X02
- removed P5: DGND, Pin_Headers:Pin_Header_Straight_1x01, symbol CONN_01X01
- removed P6: CONN_01X03, Pin_Headers:Pin_Header_Straight_1x03, symbol CONN_01X03
- added C10, C11, C12, C13, C5, C6, C8, C9: C, Capacitors_SMD:C_0805_HandSoldering, symbol C
- added C3, C4: 0.1uF, Capacitors_SMD:C_0805_HandSoldering, symbol C
- added CN2: BREAKOUT, Pin_Headers:Pin_Header_Straight_1x12, symbol BREAKOUT
- added D1: TVS DIODE, HERMESLITE:SOD323, symbol DIODESCH2
- added L1, L2, L3, L4, L5, L6, L7, L8: INDUCTOR, Choke_Toroid_ThroughHole:Choke_Toroid_6,5x13mm_Vertical, symbol INDUCTOR
- added P1: BNC, HERMESLITE:BNCRA, symbol BNC
- added P2: FLT1, Pin_Headers:Pin_Header_Straight_1x02, symbol CONN_01X02
- added P3: FLT2, Pin_Headers:Pin_Header_Straight_1x02, symbol CONN_01X02
- added P6: +S12V, Pin_Headers:Pin_Header_Straight_1x02, symbol CONN_01X02
- added U1, U2: PE4259-53, Transistors_SMD:sc70-6, symbol PE4259-53
- FB1: footprint SMD_Packages:SMD-0805 -> SMD_Packages:SMD-1206
- P5: renamed from P2; footprint Pin_Headers:Pin_Header_Straight_1x02 -> Pin_Headers:Pin_Header_Straight_2x01
- renumbered C5 to C1, C13 to C15, C14 to C16, C10 to C17, C12 to C18, C15 to C19, C4 to C2, C9 to C20, C8 to C21, C11 to C22, C3 to C23, C7 to C24, C6 to C25, D2 to D3, L1 to L10, P3 to P4, Q9 to Q10, Q8 to Q11, Q1 to Q3, Q2 to Q4, Q4 to Q5, Q5 to Q6, Q6 to Q8, Q3 to Q9, R13 to R10, R15 to R11, R14 to R12, R16 to R13, R11 to R14, R9 to R15, R7 to R16, R6 to R17, R3 to R18, R4 to R3, R5 to R4, R8 to R5, R10 to R6, R12 to R7, R17 to R8, R18 to R9, T3 to T1, T4 to T3, T5 to T4, T1 to T5
Connections:
- net labels added: GPIO0
- net labels removed: +12V, +3V, 10/12M, 160M, 17/15M, 30/20M, 60/40M, 80/75M, ANT, RX/TX, S12V
- wire segments 157 -> 207
Other:
- note added: "(<----\npopulate only if using\nexternal filter board)"
- note added: "(Band Specific Values)"
- note added: "(Omit U1/U2 and filter\ncomponents if using\nexternal filter board)"
- note added: "(populate only if using\nexternal filter board)"
- note added: "BN-43-2402 L\nBN-61-2402 H\n 6T 2x3T #30"
- note added: "Note: When not using SPI, \nGPIO0 is band select.\n\nCN2 will be removed after circuit prototype phase complete.\n\n"
- note added: "Omitted for\nlower freq's"
- note removed: "BN-43-2402\n 6T 2x3T #30"
- note removed: "S12V"
- moved on the sheet: P5
