File: frontend/basic 1w pa/basic-1W-pa - wo filters.sch (KiCad schematic (older format))
At the start: 54 parts, among them CN1 EDGE, P1 CONN_01X02, P2 CONN_02X01, P3 CONN_01X02, P5 DGND, P6 CONN_01X03, Q1 BS170, Q2 2N3906, Q3 PZT2222A, Q4 BS170, Q5 2N3904, Q6 BS170, Q7 BS170, Q8 BS170, Q9 BS170, T1 TRANSFO, T2 8:1, T3 4:1, T4 TRANSF, T5 TRANSF

Commit message: 10W amp initial commit
Parts:
- removed P2: CONN_02X01, Pin_Headers:Pin_Header_Straight_1x02, symbol CONN_02X01
- removed P5: DGND, Pin_Headers:Pin_Header_Straight_1x01, symbol CONN_01X01
- removed P6: CONN_01X03, Pin_Headers:Pin_Header_Straight_1x03, symbol CONN_01X03
- removed T1: TRANSFO, Socket_Strips:Socket_Strip_Straight_2x02, symbol TRANSFO
- added CN2: BREAKOUT, Pin_Headers:Pin_Header_Straight_1x12, symbol BREAKOUT
- added P2, P3: CONN_01X02, Pin_Headers:Pin_Header_Straight_1x02, symbol CONN_01X02
- added P6: +S12V, Pin_Headers:Pin_Header_Straight_1x02, symbol CONN_01X02
- C1: renamed from C5; footprint Capacitors_SMD:C_0805_HandSoldering -> Capacitors_SMD:C_1206_HandSoldering
- C15: renamed from C13; footprint Capacitors_SMD:C_0805_HandSoldering -> Capacitors_SMD:C_1206_HandSoldering
- C17: renamed from C10; footprint Capacitors_SMD:C_0805_HandSoldering -> Capacitors_SMD:C_1206_HandSoldering
- C18: renamed from C12; footprint Capacitors_SMD:C_0805_HandSoldering -> Capacitors_SMD:C_1206_HandSoldering
- C19: renamed from C15; footprint Capacitors_SMD:C_0805_HandSoldering -> Capacitors_SMD:C_1206_HandSoldering
- C2: renamed from C4; footprint Capacitors_SMD:C_0805_HandSoldering -> Capacitors_SMD:C_1206_HandSoldering
- C20: renamed from C9; footprint Capacitors_SMD:C_0805_HandSoldering -> Capacitors_SMD:C_1206_HandSoldering
- C21: renamed from C8; footprint Capacitors_SMD:C_0805_HandSoldering -> Capacitors_SMD:C_1206_HandSoldering
- C22: renamed from C11; footprint Capacitors_SMD:C_0805_HandSoldering -> Capacitors_SMD:C_1206_HandSoldering
- C23: renamed from C3; footprint Capacitors_SMD:C_0805_HandSoldering -> Capacitors_SMD:C_1206_HandSoldering
- C25: renamed from C6; footprint Capacitors_SMD:C_0805_HandSoldering -> Capacitors_SMD:C_1206_HandSoldering
- FB1: footprint SMD_Packages:SMD-0805 -> SMD_Packages:SMD-1206
- P1: footprint Pin_Headers:Pin_Header_Angled_1x02 -> (none)
- R1, R2: footprint Resistors_SMD:R_0805_HandSoldering -> Resistors_SMD:R_1206_HandSoldering
- R10: renamed from R13; footprint Resistors_SMD:R_0805_HandSoldering -> Resistors_SMD:R_1206_HandSoldering
- R11: renamed from R15; footprint Resistors_SMD:R_0805_HandSoldering -> Resistors_SMD:R_1206_HandSoldering
- R12: renamed from R14; footprint Resistors_SMD:R_0805_HandSoldering -> Resistors_SMD:R_1206_HandSoldering
- R13: renamed from R16; footprint Resistors_SMD:R_0805_HandSoldering -> Resistors_SMD:R_1206_HandSoldering
- R14: renamed from R11; footprint Resistors_SMD:R_0805_HandSoldering -> Resistors_SMD:R_1206_HandSoldering
- R15: renamed from R9; footprint Resistors_SMD:R_0805_HandSoldering -> Resistors_SMD:R_1206_HandSoldering
- R16: renamed from R7; footprint Resistors_SMD:R_0805_HandSoldering -> Resistors_SMD:R_1206_HandSoldering
- R17: renamed from R6; footprint Resistors_SMD:R_0805_HandSoldering -> Resistors_SMD:R_1206_HandSoldering
- R18: renamed from R3; footprint Resistors_SMD:R_0805_HandSoldering -> Resistors_SMD:R_1206_HandSoldering
- R3: renamed from R4; footprint Resistors_SMD:R_0805_HandSoldering -> Resistors_SMD:R_1206_HandSoldering
- R4: renamed from R5; footprint Resistors_SMD:R_0805_HandSoldering -> Resistors_SMD:R_1206_HandSoldering
- R5: renamed from R8; footprint Resistors_SMD:R_0805_HandSoldering -> Resistors_SMD:R_1206_HandSoldering
- R6: renamed from R10; footprint Resistors_SMD:R_0805_HandSoldering -> Resistors_SMD:R_1206_HandSoldering
- R7: renamed from R12; footprint Resistors_SMD:R_0805_HandSoldering -> Resistors_SMD:R_1206_HandSoldering
- R8: renamed from R17; footprint Resistors_SMD:R_0805_HandSoldering -> Resistors_SMD:R_1206_HandSoldering
- R9: renamed from R18; footprint Resistors_SMD:R_0805_HandSoldering -> Resistors_SMD:R_1206_HandSoldering
- renumbered C14 to C16, C7 to C24, D2 to D3, L1 to L10, P3 to P4, Q9 to Q10, Q8 to Q11, Q1 to Q3, Q2 to Q4, Q4 to Q5, Q5 to Q6, Q6 to Q8, Q3 to Q9, T3 to T1, T4 to T3, T5 to T4
Connections:
- net RX/TX is gone; now on an unnamed net: Q3.1 (D), T4.1 (S1)
- net GND: now also P1.2 (P2), P2.1 (P1), P2.2 (P2), P3.1 (P1), P3.2 (P2), P6.1 (P1)
- net PTT#: now also CN2.4 (PTT#)
- net at CN1.A13 (5V), CN1.A14 (5V), FB1.1: now also CN2.5 (5V)
- net at CN1.A17 (DGND), CN1.A18 (DGND): now also CN2.12 (DGND)
- net at CN1.B18 (SCLK): now also CN2.10 (SCLK)
- net at Q5.1 (D), R5.1, R6.2: no longer C17.1, T3.1 (S1)
- net +12V: no longer names the net of C24.1, C25.1, CN1.A11 (12V), CN1.A12 (12V), L10.2, Q4.1 (E), R4.1
- net +12V: now also CN2.6 (12V)
- net +3V: no longer names the net of CN1.A15 (3V), CN1.A16 (3V)
- net +3V: now also CN2.11 (3V)
- net 10/12M: no longer names the net of CN1.B17 (SDO)
- net 10/12M: now also CN2.9 (SDO)
- net 160M renamed GPIO0
- net GPIO0: now also CN2.3 (GPIO0)
- net 17/15M: no longer names the net of CN1.B16 (SDI)
- net 17/15M: now also CN2.8 (SDI)
- net 30/20M: no longer names the net of CN1.B15 (SEN)
- net 30/20M: now also CN2.7 (SEN)
- net 60/40M: no longer names the net of CN1.B14 (GPIO2)
- net 60/40M: now also CN2.1 (GPIO2)
- net 80/75M: no longer names the net of CN1.B13 (GPIO1)
- net 80/75M: now also CN2.2 (GPIO1)
- net S12V: no longer names the net of C20.1, Q4.3 (C), R5.2
- net S12V: now also P6.2 (P2)
- new net: C17.1, T3.1 (S1)
Other:
- note added: "BN-43-2402 L\nBN-61-2402 H\n 6T 2x3T #30"
- note added: "Note: When not using SPI, 3 GPIO signals are available. \nGPIO0 is band select.\nIf SPI is used, GPIO2 becomes SEN1 (Transmit Strobe - Alex Protocol)\nSEN should be called SEN0 (Receive Strobe - Alex Protocol)\n"
- note added: "Omitted for\nlower freq's"
- note added: "To/from Filters"
- note removed: "BN-43-2402\n 6T 2x3T #30"
- note removed: "BN-61-2402\n 2x4T #30"
- note removed: "Ground\nOption"
- note removed: "S12V"
