File: frontend/basic 10w pa/Filter1.sch (KiCad schematic (older format))
At the start: 62 parts, among them K10 D3002, K11 D3002, K12 D3002, K13 D3002, K2 D3002, K3 D3002, K4 D3002, K5 D3002, K6 D3002, K7 D3002, K8 D3002, K9 D3002, P4 CONN_01X07, U1 ULN2003A

Commit message: Cleanup BOM
Parts:
- removed P4: CONN_01X07, Pin_Headers:Pin_Header_Straight_1x07, symbol CONN_01X07
- added P4: CONN_01X08, Pin_Headers:Pin_Header_Straight_1x08, symbol CONN_01X08
- renumbered C21 to C17, C17 to C18, C18 to C19, C19 to C20, C20 to C21, C27 to C23, C23 to C24, C24 to C25, C25 to C26, C26 to C27, C33 to C29, C29 to C30, C30 to C31, C31 to C32, C32 to C33, C39 to C35, C35 to C36, C36 to C37, C37 to C38, C38 to C39, K2 to K1, K3 to K2, K4 to K3, K5 to K4, K6 to K5, K7 to K6, K8 to K7, K13 to K8, L9 to L10, L10 to L11, L11 to L12, L12 to L13, L19 to L15, L15 to L16, L16 to L17, L17 to L18, L18 to L19, L25 to L21, L21 to L22, L22 to L23, L23 to L24, L24 to L25, L7 to L3, L3 to L4, L4 to L5, L5 to L6, L6 to L7, L13 to L9
Connections:
- net GND: now also P4.8 (P8)
- net at U1.10 (O7): now also P4.7 (P7)
- net at K12.10 (-), K6.10 (-), U1.11 (O6): now also P4.6 (P6)
- net at K11.10 (-), K5.10 (-), U1.12 (O5): now also P4.5 (P5)
- net at K10.10 (-), K4.10 (-), U1.13 (O4): now also P4.4 (P4)
- net at K3.10 (-), K9.10 (-), U1.14 (O3): now also P4.3 (P3)
- net at K2.10 (-), K8.10 (-), U1.15 (O2): now also P4.2 (P2)
- net at K1.10 (-), K7.10 (-), U1.16 (O1): now also P4.1 (P1)
- net +PTT: now reaches U1.7 (I7)
Other:
- note added: "/PTT"
