File: frontend/basic 10w pa/basic-10W-pa.sch (KiCad schematic (older format))
At the start: 43 parts, among them CN1 EDGE, K1 D3002, P1 CONN_01X02, P2 CONN_02X01, P3 CONN_01X02, P5 DGND, P6 CONN_01X03, Q1 2N3906, Q2 2N3906, Q3 RD16HHF1, Q4 RD16HHF1, T1 TRANSFO, T2 8:1, T3 4:1, T4 TRANSF

Commit message: Cleanup BOM
Parts:
- removed Q3, Q4: RD16HHF1, symbol MOSFET_N
- added L26, L27: 68nH, SMD_Packages:SMD-0805, symbol INDUCTOR_SMALL
- added P7: CONN_01X03, Pin_Headers:Pin_Header_Straight_1x03, symbol CONN_01X03
- added Q3, Q4: RD16HHF1, Transistors_TO-220:TO-220_Neutral123_Vertical_LargePads, symbol RD16HHF1
- D1: footprint (none) -> Diodes_SMD:Diode-SMA_Handsoldering
- K13: renamed from K1; footprint (none) -> Sockets_DIP:DIP-10__300
- L1: footprint (none) -> Choke_Axial_ThroughHole:Choke_Horizontal_RM10mm
- P6: footprint (none) -> Pin_Headers:Pin_Header_Straight_1x03
- Q1, Q2: footprint (none) -> Transistors_SMD:sot23
- T4: footprint (none) -> HERMESLITE:TRANSF
- VR1, VR2: footprint (none) -> Potentiometers:Potentiometer_Bourns_3296W_3-8Zoll_Inline_ScrewUp
Connections:
- net ANT: now also K13.4 (R1), P7.2 (P2); no longer K13.3 (C1), T1.4 (SB)
- net GND: now also Q3.2 (S), Q4.2 (S)
- net at C8.2, R2.1: now also L26.2
- net at R7.1, T4.5 (P5): now also Q3.3 (D)
- net at C12.1, R8.1, T4.4 (P4): now also Q4.3 (D)
- net at C9.2, R4.1: now also L27.2
- net +PTT: now reaches Q2.3 (C), R6.1
- net at K13.2 (T1), P6.3 (P3): now also P7.1 (P1)
- new net: K13.3 (C1), T1.4 (SB)
- new net: L26.1, Q3.1 (G)
- new net: L27.1, Q4.1 (G)
Other:
- note added: "This jumper pair selects whether the TX signal \nuses or bypasses the BPF. Jumpers connect \n1/2 or 2/3 on both at same time. This insures that\nBPF is completely out of circuit during TX when BPF \nbypass is active."
- note removed: "This jumper selects whether the TX signal \nuses or bypasses the BPF."
