File: frontend/basic 10w pa/basic-10W-pa.kicad_pcb (KiCad board)
At the start: 2 copper layers, 115 x 126.8 mm, 121 parts, among them CN1 EDGE, K1 D3002, K10 D3002, K11 D3002, K12 D3002, K2 D3002, K3 D3002, K4 D3002, K5 D3002, K6 D3002, K7 D3002, K8 D3002, K9 D3002, P1 CONN_01X02, P2 CONN_02X01, P3 CONN_01X02, P4 CONN_01X07, P5 DGND, P6 CONN_01X03, Q1 BS170, Q2 2N3906, Q3 PZT2222A, Q4 BS170, Q5 2N3904, Q6 BS170, Q7 BS170, Q8 BS170, Q9 BS170, T1 TRANSFO, T2 8:1, T3 4:1, T4 TRANSF, T5 TRANSF, U1 ULN2003A

Commit message: Beginning updates for RD16HHF1 design
Parts:
- removed D2: 1N4003, Diodes_SMD:Diode-SMB_Handsoldering
- removed MH1, MH2, MH3, MH4, MH5: VAL**, HERMESLITE:MH
- removed Q5: 2N3904, Transistors_SMD:sot23
- removed Q6, Q7, Q8, Q9: BS170, Housings_TO-92:TO-92-Free-inline-wide
- removed R10: 2.21k, Resistors_SMD:R_0805_HandSoldering
- removed R11: 68.1, Resistors_SMD:R_0805_HandSoldering
- removed R12: 33.2, Resistors_SMD:R_0805_HandSoldering
- removed R13, R14, R18: 221, Resistors_SMD:R_0805_HandSoldering
- removed R15, R16: 2.21, Resistors_SMD:R_0805_HandSoldering
- removed R17: 22.1k, Resistors_SMD:R_0805_HandSoldering
- removed R9: 56.2, Resistors_SMD:R_0805_HandSoldering
- removed T5: TRANSF, HERMESLITE:TRANSF
- added C1: 0.1uF, Capacitors_SMD:C_0805_HandSoldering, F.Cu at (171.1, 161.2)
- added C2: 0.1uF, Capacitors_SMD:C_0805_HandSoldering, F.Cu at (169.5, 153.9)
- added D1: 1N5231, Diodes_SMD:Diode-SMA_Handsoldering, F.Cu at (180.0, 140.6)
- added K13: D3002, Sockets_DIP:DIP-10__300, F.Cu at (123.6, 155.5)
- added L26: 68nH, SMD_Packages:SMD-0805, F.Cu at (178.9, 147.5)
- added L27: 68nH, SMD_Packages:SMD-0805, F.Cu at (178.9, 151.4)
- added P7: CONN_01X03, Pin_Headers:Pin_Header_Straight_1x03, F.Cu at (156.0, 161.7)
- added VR1: 1k MT, Potentiometers:Potentiometer_Bourns_3296W_3-8Zoll_Inline_ScrewUp, F.Cu at (143.3, 159.8)
- added VR2: 1K MT, Potentiometers:Potentiometer_Bourns_3296W_3-8Zoll_Inline_ScrewUp, F.Cu at (150.1, 157.7)
- C10, C8: value 0.01uF -> 0.1uF
- C11: value 220pF -> 0.1uF
- C12: value 0.01uF -> 3300pF
- C13: value 0.01uF -> 4700pF
- C14: value 47uF 16V -> 0.1uF; footprint Discret:C1V8 -> Capacitors_SMD:C_0805_HandSoldering
- L1: value INDUCTOR -> FT50-43 10T #26
- P4: value CONN_01X07 -> CONN_01X08; footprint Pin_Headers:Pin_Header_Straight_1x07 -> Pin_Headers:Pin_Header_Straight_1x08
- Q1: value BS170 -> 2N3906; footprint Housings_TO-92:TO-92-Free-inline-wide -> Transistors_SMD:sot23
- Q3: value PZT2222A -> RD16HHF1; footprint SMD_Packages:SOT-223 -> Transistors_TO-220:TO-220_Neutral123_Vertical_LargePads
- Q4: value BS170 -> RD16HHF1; footprint Housings_TO-92:TO-92-Free-inline-wide -> Transistors_TO-220:TO-220_Neutral123_Vertical_LargePads
- R1: value 4.99k -> 1k
- R2: value 22.1k -> 47
- R4: value 4.99k -> 47
- R6: value 2.21k -> 220
- R7: value 475 -> 470 .5W
- R8: value 22.1 -> 470
- moved P6 96.3 mm to (199.5, 40.0)
- moved T4 79.0 mm to (197.6, 49.9)
- moved Q3 42.1 mm to (154.4, 51.7)
- moved Q4 15.2 mm to (153.8, 42.9)
Connections:
- C10 pad 2: GND -> Net-(C10-Pad2)
- C13 pad 1: Net-(C13-Pad1) -> GND
- C13 pad 2: GND -> +12V
- C14 pad 1: Net-(C13-Pad1) -> GND
- C14 pad 2: GND -> +12V
- C15 pad 1: Net-(C12-Pad1) -> GND
- C15 pad 2: GND -> +12V
- C8 pad 1: Net-(C8-Pad1) -> Net-(C10-Pad2)
- C9 pad 1: S12V -> Net-(C11-Pad2)
- C9 pad 2: GND -> Net-(C9-Pad2)
- L1 pad 1: Net-(C13-Pad1) -> +12V
- L1 pad 2: +12V -> Net-(L1-Pad2)
- P4 pad 7: GND -> Net-(P4-Pad7)
- P6 pad 1: PTT# -> Net-(K13-Pad9)
- P6 pad 3: GND -> Net-(K13-Pad2)
- Q1 pad 1: RX/TX -> +12V
- Q1 pad 2: Net-(C3-Pad1) -> Net-(Q1-Pad2)
- Q1 pad 3: Net-(Q1-Pad3) -> Net-(K13-Pad1)
- Q2 pad 3: S12V -> +PTT
- Q3 pad 1: Net-(C8-Pad1) -> Net-(L26-Pad1)
- Q3 pad 2: Net-(Q3-Pad2) -> GND
- Q3 pad 3: Net-(C11-Pad2) -> Net-(Q3-Pad3)
- Q4 pad 1: Net-(C10-Pad1) -> Net-(L27-Pad1)
- Q4 pad 2: Net-(D2-Pad1) -> GND
- Q4 pad 3: Net-(P6-Pad2) -> Net-(C12-Pad1)
- R1 pad 1: Net-(C3-Pad1) -> Net-(Q1-Pad2)
- R2 pad 1: Net-(C3-Pad1) -> Net-(C8-Pad2)
- R2 pad 2: GND -> Net-(C1-Pad1)
- R4 pad 1: PTT# -> Net-(C9-Pad2)
- R4 pad 2: Net-(Q2-Pad2) -> Net-(C2-Pad1)
- R5 pad 1: +12V -> Net-(Q2-Pad2)
- R5 pad 2: Net-(Q2-Pad2) -> PTT#
- R6 pad 1: Net-(Q3-Pad2) -> +PTT
- R6 pad 2: Net-(C8-Pad1) -> Net-(C3-Pad1)
- R7 pad 1: Net-(C8-Pad1) -> Net-(Q3-Pad3)
- R7 pad 2: GND -> Net-(C10-Pad1)
- R8 pad 1: Net-(C10-Pad1) -> Net-(C12-Pad1)
- R8 pad 2: S12V -> Net-(C11-Pad1)
- T1 pad 4: ANT -> Net-(K13-Pad3)
- T2 pad 1: Net-(Q1-Pad3) -> Net-(K13-Pad7)
- T3 pad 1: Net-(C8-Pad2) -> Net-(C10-Pad2)
- T3 pad 2: GND -> Net-(C11-Pad2)
- T4 pad 1: Net-(C10-Pad1) -> Net-(P6-Pad2)
- T4 pad 2: Net-(Q3-Pad2) -> GND
- T4 pad 3: Net-(C12-Pad1) -> Net-(L1-Pad2)
- T4 pad 4: Net-(Q6-Pad2) -> Net-(C12-Pad1)
- T4 pad 5: Net-(Q7-Pad2) -> Net-(Q3-Pad3)
- T4 pad 6: Net-(C12-Pad1) -> Net-(L1-Pad2)
- U1 pad 10: Net-(U1-Pad10) -> Net-(P4-Pad7)
- U1 pad 7: Net-(U1-Pad7) -> +PTT
Routing:
- net GND: track 831.2 -> 601.3 mm, vias 10 -> 7
- net RX/TX: track 180.1 -> 7.62 mm, vias 6 -> 0
- net Net-(C12-Pad1): track 91.8 -> 0.00 mm, vias 2 -> 0
- net Net-(Q6-Pad2): track 74.7 -> 0.00 mm, vias 1 -> 0
- net Net-(P6-Pad2): track 73.2 -> 0.80 mm, vias 8 -> 0
- net Net-(C10-Pad1): track 66.9 -> 0.00 mm
- net Net-(Q7-Pad2): track 55.2 -> 0.00 mm
- net Net-(Q2-Pad2): track 50.5 -> 0.00 mm, vias 3 -> 0
- net Net-(Q7-Pad1): track 48.6 -> 0.00 mm, vias 2 -> 0
- net +12V: track 330.1 -> 293.5 mm, vias 3 -> 2
- net Net-(C13-Pad1): track 31.5 -> 0.00 mm
- net PTT#: track 61.3 -> 30.0 mm, vias 3 -> 1
- net Net-(Q6-Pad3): track 25.2 -> 0.00 mm, vias 2 -> 0
- net Net-(Q6-Pad1): track 23.6 -> 0.00 mm, vias 1 -> 0
- net Net-(Q7-Pad3): track 21.9 -> 0.00 mm, vias 1 -> 0
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Other:
- outline, holes or cut-outs redrawn
