File: frontend/new 10w pa/TX-filter.sch (KiCad schematic (older format))
At the start: 50 parts, among them K2 D3002, K3 D3002, K4 D3002, K5 D3002, K6 D3002, P8 CONN_01X07, U3 TPIC6B595, U4 TPIC6B595

Commit message: Minor updates to v1.12
Parts:
- removed P8: CONN_01X07, Pin_Headers:Pin_Header_Straight_1x07, symbol CONN_01X07
- added P8: CONN_01X08, Pin_Headers:Pin_Header_Straight_1x07, symbol CONN_01X08
Connections:
- net labels added: ANT1, ANT2, ANT3
- wire segments 200 -> 206
- no-connect marks 9 -> 6
Other:
- note added: "10/12M\n17/15M\n30/20M\n60/40M\n80/75M\n160M\n/PTT"
- moved on the sheet: C15, C16, C17, C18, C19, C20, C21, C22, C23, C24, C25, C26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

Commit message: Starting Layout
Parts:
- P8: footprint Pin_Headers:Pin_Header_Straight_1x07 -> Pin_Headers:Pin_Header_Straight_1x08
Changed lines of the file:
@@
 F 0 "P8" H 1700 5450 50  0000 C CNN
 F 1 "CONN_01X08" V 1800 5000 50  0000 C CNN
-F 2 "Pin_Headers:Pin_Header_Straight_1x07" H 1700 5000 60  0001 C CNN
+F 2 "Pin_Headers:Pin_Header_Straight_1x08" H 1700 5000 60  0001 C CNN
 F 3 "" H 1700 5000 60  0000 C CNN
 	1    1700 5000

Commit message: Continuing board routing
Parts:
- removed D2: RED, LEDs:LED-1206, symbol LED
- removed D3: YEL, LEDs:LED-1206, symbol LED
- removed R11, R12: 1k, Resistors_SMD:R_0805, symbol R
- C15, C16, C17, C18, C19, C20, C21, C22, C23, C24, C25, C26, C27, C28, C29, C30, C31, C32, C33, C34, C35, C36, C37, C38, C39, C40, C41, C42: footprint Capacitors_SMD:C_0805 -> HERMESLITE:C_0805
- K2, K3, K4, K5, K6: footprint Sockets_DIP:DIP-10__300 -> HERMESLITE:D3002
Connections:
- wire segments 206 -> 198
- no-connect marks 6 -> 8

Commit message: Minor filter updates
Parts:
- added C80, C81: 150pF, HERMESLITE:C_0805, symbol C
- C16, C39: value 300pF -> 150pF
Connections:
- net GND: now also C80.2, C81.2
Other:
- moved on the sheet: C16, C22, C28, C33, C39, L10, L5
Changed lines of the file:
@@
 	3900 4650 1900 4650
 Wire Wire Line
-	1900 4750 3800 4750
-Wire Wire Line
-	1900 4850 3700 4850
+	3800 4750 1900 4750
+Wire Wire Line
+	3700 4850 1900 4850
 Wire Wire Line
 	1900 5050 4000 5050
@@
 L INDUCTOR L5
 U 1 1 54A1CC07
-P 6200 1850
-F 0 "L5" V 6150 1850 40  0000 C CNN
-F 1 "300nH" V 6300 1850 40  0000 C CNN
-F 2 "Choke_Toroid_ThroughHole:Choke_Toroid_6,5x13mm_Vertical" H 6200 1850 60  0001 C CNN
-F 3 "" H 6200 1850 60  0000 C CNN
-	1    6200 1850
+P 6400 1850
+F 0 "L5" V 6350 1850 40  0000 C CNN
+F 1 "300nH" V 6500 1850 40  0000 C CNN
+F 2 "Choke_Toroid_ThroughHole:Choke_Toroid_6,5x13mm_Vertical" H 6400 1850 60  0001 C CNN
+F 3 "" H 6400 1850 60  0000 C CNN
+	1    6400 1850
 	0    -1   -1   0
 $EndComp
@@
 L C C28
 U 1 1 54A1CC0D
-P 6650 2050
-F 0 "C28" H 6650 2150 40  0000 L CNN
-F 1 "560pF" H 6400 1950 40  0000 L CNN
-F 2 "HERMESLITE:C_0805" H 6688 1900 30  0001 C CNN
-F 3 "" H 6650 2050 60  0000 C CNN
-	1    6650 2050
+P 6850 2050
+F 0 "C28" H 6850 2150 40  0000 L CNN
+F 1 "560pF" H 6600 1950 40  0000 L CNN
+F 2 "HERMESLITE:C_0805" H 6888 1900 30  0001 C CNN
+F 3 "" H 6850 2050 60  0000 C CNN
+	1    6850 2050
 	1    0    0    -1
 $EndComp
@@
 L INDUCTOR L10
 U 1 1 54A1CC13
-P 7100 1850
-F 0 "L10" V 7050 1850 40  0000 C CNN
-F 1 "300nH" V 7200 1850 40  0000 C CNN
-F 2 "Choke_Toroid_ThroughHole:Choke_Toroid_6,5x13mm_Vertical" H 7100 1850 60  0001 C CNN
-F 3 "" H 7100 1850 60  0000 C CNN
-	1    7100 1850
+P 7300 1850
+F 0 "L10" V 7250 1850 40  0000 C CNN
+F 1 "300nH" V 7400 1850 40  0000 C CNN
+F 2 "Choke_Toroid_ThroughHole:Choke_Toroid_6,5x13mm_Vertical" H 7300 1850 60  0001 C CNN
+F 3 "" H 7300 1850 60  0000 C CNN
+	1    7300 1850
 	0    -1   -1   0
 $EndComp
@@
 L C C39
 U 1 1 54A1CC19
-P 7550 2050
-F 0 "C39" H 7550 2150 40  0000 L CNN
-F 1 "300pF" H 7350 1950 40  0000 L CNN
-F 2 "HERMESLITE:C_0805" H 7588 1900 30  0001 C CNN
-F 3 "" H 7550 2050 60  0000 C CNN
-	1    7550 2050
+P 7750 2050
+F 0 "C39" H 7750 2150 40  0000 L CNN
+F 1 "150pF" H 7550 1950 40  0000 L CNN
+F 2 "HERMESLITE:C_0805" H 7788 1900 30  0001 C CNN
+F 3 "" H 7750 2050 60  0000 C CNN
+	1    7750 2050
 	1    0    0    -1
 $EndComp
@@
 L GND #PWR034
 U 1 1 54A1CC1F
-P 6650 2250
-F 0 "#PWR034" H 6650 2250 30  0001 C CNN
-F 1 "GND" H 6650 2180 30  0001 C CNN
-F 2 "" H 6650 2250 60  0000 C CNN
-F 3 "" H 6650 2250 60  0000 C CNN
-	1    6650 2250
+P 6850 2250
+F 0 "#PWR034" H 6850 2250 30  0001 C CNN
+F 1 "GND" H 6850 2180 30  0001 C CNN
+F 2 "" H 6850 2250 60  0000 C CNN
+F 3 "" H 6850 2250 60  0000 C CNN
+	1    6850 2250
 	1    0    0    -1
 $EndComp
@@
 L GND #PWR035
 U 1 1 54A1CC25
-P 5750 2250
-F 0 "#PWR035" H 5750 2250 30  0001 C CNN
-F 1 "GND" H 5750 2180 30  0001 C CNN
-F 2 "" H 5750 2250 60  0000 C CNN
-F 3 "" H 5750 2250 60  0000 C CNN
-	1    5750 2250
+P 5950 2250
+F 0 "#PWR035" H 5950 2250 30  0001 C CNN
+F 1 "GND" H 5950 2180 30  0001 C CNN
+F 2 "" H 5950 2250 60  0000 C CNN
+F 3 "" H 5950 2250 60  0000 C CNN
+	1    5950 2250
 	1    0    0    -1
 $EndComp
@@
 L GND #PWR036
 U 1 1 54A1CC2B
-P 7550 2250
-F 0 "#PWR036" H 7550 2250 30  0001 C CNN
-F 1 "GND" H 7550 2180 30  0001 C CNN
-F 2 "" H 7550 2250 60  0000 C CNN
-F 3 "" H 7550 2250 60  0000 C CNN
-	1    7550 2250
-	1    0    0    -1
-$EndComp
-Text Notes 6100 2400 0    60   ~ 0
+P 7750 2250
+F 0 "#PWR036" H 7750 2250 30  0001 C CNN
+F 1 "GND" H 7750 2180 30  0001 C CNN
+F 2 "" H 7750 2250 60  0000 C CNN
+F 3 "" H 7750 2250 60  0000 C CNN
+	1    7750 2250
+	1    0    0    -1
+$EndComp
+Text Notes 6300 2400 0    60   ~ 0
 17/15M
 Wire Wire Line
-	6500 1850 6800 1850
-Connection ~ 6650 1850
-Connection ~ 6800 1850
-Connection ~ 7400 1850
-Wire Wire Line
-	5300 1850 5900 1850
+	6700 1850 7000 1850
+Connection ~ 6850 1850
+Connection ~ 7000 1850
+Connection ~ 7600 1850
+Wire Wire Line
+	5300 1850 6100 1850
 $Comp
 L C C16
 U 1 1 54A1CC37
-P 5750 2050
-F 0 "C16" H 5750 2150 40  0000 L CNN
-F 1 "300pF" H 5500 1950 40  0000 L CNN
-F 2 "HERMESLITE:C_0805" H 5788 1900 30  0001 C CNN
-F 3 "" H 5750 2050 60  0000 C CNN
-	1    5750 2050
-	1    0    0    -1
-$EndComp
-Wire Wire Line
-	7400 1850 7800 1850
-Wire Wire Line
-	7800 1850 7800 2450
-Wire Wire Line
-	7800 2450 5500 2450
+P 5950 2050
+F 0 "C16" H 5950 2150 40  0000 L CNN
+F 1 "150pF" H 6000 1900 40  0000 L CNN
+F 2 "HERMESLITE:C_0805" H 5988 1900 30  0001 C CNN
+F 3 "" H 5950 2050 60  0000 C CNN
+	1    5950 2050
+	1    0    0    -1
+$EndComp
+Wire Wire Line
+	7600 1850 8150 1850
+Wire Wire Line
+	8150 1850 8150 2450
+Wire Wire Line
+	8150 2450 5500 2450
 Wire Wire Line
 	5500 2450 5500 2150
 Wire Wire Line
 	5500 2150 5300 2150
-Connection ~ 7550 1850
-Connection ~ 5750 1850
-Text Notes 7000 1750 2    50   ~ 0
+Connection ~ 7750 1850
+Connection ~ 5950 1850
+Text Notes 7200 1750 2    50   ~ 0
 T37-6 10T #26
 $Comp
@@
 L C C22
 U 1 1 54A56D23
-P 6200 2050
-F 0 "C22" V 6150 2150 40  0000 L CNN
-F 1 "DNI" V 6050 1950 40  0000 L CNN
-F 2 "HERMESLITE:C_0805" H 6238 1900 30  0001 C CNN
-F 3 "" H 6200 2050 60  0000 C CNN
-	1    6200 2050
+P 6400 2050
+F 0 "C22" V 6350 2150 40  0000 L CNN
+F 1 "DNI" V 6250 1950 40  0000 L CNN
+F 2 "HERMESLITE:C_0805" H 6438 1900 30  0001 C CNN
+F 3 "" H 6400 2050 60  0000 C CNN
+	1    6400 2050
 	0    -1   -1   0
 $EndComp
@@
 L C C33
 U 1 1 54A56D84
-P 7100 2050
-F 0 "C33" V 7050 2150 40  0000 L CNN
-F 1 "DNI" V 6950 1950 40  0000 L CNN
-F 2 "HERMESLITE:C_0805" H 7138 1900 30  0001 C CNN
-F 3 "" H 7100 2050 60  0000 C CNN
-	1    7100 2050
-	0    -1   -1   0
-$EndComp
-Wire Wire Line
-	7400 1850 7400 2050
-Wire Wire Line
-	7400 2050 7300 2050
-Wire Wire Line
-	6900 2050 6800 2050
-Wire Wire Line
-	6800 2050 6800 1850
-Wire Wire Line
-	6500 1850 6500 2050
-Wire Wire Line
-	6500 2050 6400 2050
-Wire Wire Line
-	6000 2050 5900 2050
-Wire Wire Line
-	5900 2050 5900 1850
+P 7300 2050
+F 0 "C33" V 7250 2150 40  0000 L CNN
+F 1 "DNI" V 7150 1950 40  0000 L CNN
+F 2 "HERMESLITE:C_0805" H 7338 1900 30  0001 C CNN
+F 3 "" H 7300 2050 60  0000 C CNN
+	1    7300 2050
+	0    -1   -1   0
+$EndComp
+Wire Wire Line
+	7600 1850 7600 2050
+Wire Wire Line
+	7600 2050 7500 2050
+Wire Wire Line
+	7100 2050 7000 2050
+Wire Wire Line
+	7000 2050 7000 1850
+Wire Wire Line
+	6700 1850 6700 2050
+Wire Wire Line
+	6700 2050 6600 2050
+Wire Wire Line
+	6200 2050 6100 2050
+Wire Wire Line
+	6100 2050 6100 1850
 $Comp
 L C C21
@@
 	3450 1100 4500 1100
 Wire Wire Line
-	4500 1300 3350 1300
+	3350 1300 4500 1300
 Connection ~ 3350 1300
 Wire Wire Line
@@
 	4350 4900 4500 4900
 Wire Wire Line
-	3350 1300 3350 1000
+	3350 1000 3350 1300
 Wire Wire Line
 	4100 1300 4100 5100
@@
 Connection ~ 3900 3800
 Wire Wire Line
-	3800 4750 3800 2350
+	3800 2350 3800 4750
 Wire Wire Line
 	3800 2350 4500 2350
@@
 NoConn ~ 2350 3500
 NoConn ~ 2350 1800
+$Comp
+L C C80
+U 1 1 54ABE597
+P 5750 2050
+F 0 "C80" H 5750 2150 40  0000 L CNN
+F 1 "150pF" H 5550 1900 40  0000 L CNN
+F 2 "HERMESLITE:C_0805" H 5788 1900 30  0001 C CNN
+F 3 "" H 5750 2050 60  0000 C CNN
+	1    5750 2050
+	1    0    0    -1
+$EndComp
+$Comp
+L GND #PWR044
+U 1 1 54ABE5DE
+P 5750 2250
+F 0 "#PWR044" H 5750 2250 30  0001 C CNN
+F 1 "GND" H 5750 2180 30  0001 C CNN
+F 2 "" H 5750 2250 60  0000 C CNN
+F 3 "" H 5750 2250 60  0000 C CNN
+	1    5750 2250
+	1    0    0    -1
+$EndComp
+$Comp
+L C C81
+U 1 1 54ABE696
+P 8000 2050
+F 0 "C81" H 8000 2150 40  0000 L CNN
+F 1 "150pF" H 7800 1950 40  0000 L CNN
+F 2 "HERMESLITE:C_0805" H 8038 1900 30  0001 C CNN
+F 3 "" H 8000 2050 60  0000 C CNN
+	1    8000 2050
+	1    0    0    -1
+$EndComp
+$Comp
+L GND #PWR045
+U 1 1 54ABE6E0
+P 8000 2250
+F 0 "#PWR045" H 8000 2250 30  0001 C CNN
+F 1 "GND" H 8000 2180 30  0001 C CNN
+F 2 "" H 8000 2250 60  0000 C CNN
+F 3 "" H 8000 2250 60  0000 C CNN
+	1    8000 2250
+	1    0    0    -1
+$EndComp
 $EndSCHEMATC

Commit message: Continuing routing
Connections:
- net at C33.2, C39.1, K3.4 (T1)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: now also C81.1
- net at C16.1, C22.1, K3.7 (T2)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: now also C80.1
Changed lines of the file:
@@
 	1    0    0    -1
 $EndComp
+Connection ~ 8000 1850
+Connection ~ 5750 1850
 $EndSCHEMATC

Commit message: More pcb changes
Parts:
- added C82: 0.1uF, HERMESLITE:C_0805, symbol C
Connections:
- net TXIN: now also C82.2; no longer K2.8 (C2)
- new net: C82.1, K2.8 (C2)
Changed lines of the file:
@@
 $EndComp
 $Comp
-L GND #PWR023
+L GND #PWR024
 U 1 1 5496A449
 P 6850 4150
-F 0 "#PWR023" H 6850 4150 30  0001 C CNN
+F 0 "#PWR024" H 6850 4150 30  0001 C CNN
 F 1 "GND" H 6850 4080 30  0001 C CNN
 F 2 "" H 6850 4150 60  0000 C CNN
@@
 $EndComp
 $Comp
-L GND #PWR024
+L GND #PWR025
 U 1 1 5496A44A
 P 5750 4150
-F 0 "#PWR024" H 5750 4150 30  0001 C CNN
+F 0 "#PWR025" H 5750 4150 30  0001 C CNN
 F 1 "GND" H 5750 4080 30  0001 C CNN
 F 2 "" H 5750 4150 60  0000 C CNN
@@
 $EndComp
 $Comp
-L GND #PWR025
+L GND #PWR026
 U 1 1 5496A44B
 P 7750 4150
-F 0 "#PWR025" H 7750 4150 30  0001 C CNN
+F 0 "#PWR026" H 7750 4150 30  0001 C CNN
 F 1 "GND" H 7750 4080 30  0001 C CNN
 F 2 "" H 7750 4150 60  0000 C CNN
@@
 	5400 4400 4400 4400
 $Comp
-L GND #PWR026
+L GND #PWR027
 U 1 1 5496A47D
 P 1900 5550
-F 0 "#PWR026" H 1900 5550 30  0001 C CNN
+F 0 "#PWR027" H 1900 5550 30  0001 C CNN
 F 1 "GND" H 1900 5480 30  0001 C CNN
 F 2 "" H 1900 5550 50  0000 C CNN
@@
 $EndComp
 $Comp
-L GND #PWR027
+L GND #PWR028
 U 1 1 54A155CF
 P 6800 5300
-F 0 "#PWR027" H 6800 5300 30  0001 C CNN
+F 0 "#PWR028" H 6800 5300 30  0001 C CNN
 F 1 "GND" H 6800 5230 30  0001 C CNN
 F 2 "" H 6800 5300 60  0000 C CNN
@@
 $EndComp
 $Comp
-L GND #PWR028
+L GND #PWR029
 U 1 1 54A1568D
 P 7400 5300
-F 0 "#PWR028" H 7400 5300 30  0001 C CNN
+F 0 "#PWR029" H 7400 5300 30  0001 C CNN
 F 1 "GND" H 7400 5230 30  0001 C CNN
 F 2 "" H 7400 5300 60  0000 C CNN
@@
 $EndComp
 $Comp
-L GND #PWR029
+L GND #PWR030
 U 1 1 54A171EB
 P 5950 6400
-F 0 "#PWR029" H 5950 6400 30  0001 C CNN
+F 0 "#PWR030" H 5950 6400 30  0001 C CNN
 F 1 "GND" H 5950 6330 30  0001 C CNN
 F 2 "" H 5950 6400 60  0000 C CNN
@@
 $EndComp
 $Comp
-L GND #PWR030
+L GND #PWR031
 U 1 1 54A171F1
 P 6550 6400
-F 0 "#PWR030" H 6550 6400 30  0001 C CNN
+F 0 "#PWR031" H 6550 6400 30  0001 C CNN
 F 1 "GND" H 6550 6330 30  0001 C CNN
 F 2 "" H 6550 6400 60  0000 C CNN
@@
 $EndComp
 $Comp
-L GND #PWR031
+L GND #PWR032
 U 1 1 54A1B96C
 P 6650 3200
-F 0 "#PWR031" H 6650 3200 30  0001 C CNN
+F 0 "#PWR032" H 6650 3200 30  0001 C CNN
 F 1 "GND" H 6650 3130 30  0001 C CNN
 F 2 "" H 6650 3200 60  0000 C CNN
@@
 $EndComp
 $Comp
-L GND #PWR032
+L GND #PWR033
 U 1 1 54A1B972
 P 5750 3200
-F 0 "#PWR032" H 5750 3200 30  0001 C CNN
+F 0 "#PWR033" H 5750 3200 30  0001 C CNN
 F 1 "GND" H 5750 3130 30  0001 C CNN
 F 2 "" H 5750 3200 60  0000 C CNN
@@
 $EndComp
 $Comp
-L GND #PWR033
+L GND #PWR034
 U 1 1 54A1B978
 P 7550 3200
-F 0 "#PWR033" H 7550 3200 30  0001 C CNN
+F 0 "#PWR034" H 7550 3200 30  0001 C CNN
 F 1 "GND" H 7550 3130 30  0001 C CNN
 F 2 "" H 7550 3200 60  0000 C CNN
@@
 $EndComp
 $Comp
-L GND #PWR034
+L GND #PWR035
 U 1 1 54A1CC1F
 P 6850 2250
-F 0 "#PWR034" H 6850 2250 30  0001 C CNN
+F 0 "#PWR035" H 6850 2250 30  0001 C CNN
 F 1 "GND" H 6850 2180 30  0001 C CNN
 F 2 "" H 6850 2250 60  0000 C CNN
@@
 $EndComp
 $Comp
-L GND #PWR035
+L GND #PWR036
 U 1 1 54A1CC25
 P 5950 2250
-F 0 "#PWR035" H 5950 2250 30  0001 C CNN
+F 0 "#PWR036" H 5950 2250 30  0001 C CNN
 F 1 "GND" H 5950 2180 30  0001 C CNN
 F 2 "" H 5950 2250 60  0000 C CNN
@@
 $EndComp
 $Comp
-L GND #PWR036
+L GND #PWR037
 U 1 1 54A1CC2B
 P 7750 2250
-F 0 "#PWR036" H 7750 2250 30  0001 C CNN
+F 0 "#PWR037" H 7750 2250 30  0001 C CNN
 F 1 "GND" H 7750 2180 30  0001 C CNN
 F 2 "" H 7750 2250 60  0000 C CNN
@@
 $EndComp
 $Comp
-L GND #PWR037
+L GND #PWR038
 U 1 1 54A1CDA5
 P 6650 1300
-F 0 "#PWR037" H 6650 1300 30  0001 C CNN
+F 0 "#PWR038" H 6650 1300 30  0001 C CNN
 F 1 "GND" H 6650 1230 30  0001 C CNN
 F 2 "" H 6650 1300 60  0000 C CNN
@@
 $EndComp
 $Comp
-L GND #PWR038
+L GND #PWR039
 U 1 1 54A1CDAB
 P 5750 1300
-F 0 "#PWR038" H 5750 1300 30  0001 C CNN
+F 0 "#PWR039" H 5750 1300 30  0001 C CNN
 F 1 "GND" H 5750 1230 30  0001 C CNN
 F 2 "" H 5750 1300 60  0000 C CNN
@@
 $EndComp
 $Comp
-L GND #PWR039
+L GND #PWR040
 U 1 1 54A1CDB1
 P 7550 1300
-F 0 "#PWR039" H 7550 1300 30  0001 C CNN
+F 0 "#PWR040" H 7550 1300 30  0001 C CNN
 F 1 "GND" H 7550 1230 30  0001 C CNN
 F 2 "" H 7550 1300 60  0000 C CNN
@@
 	1900 2450 1900 2500
 $Comp
-L GND #PWR040
+L GND #PWR041
 U 1 1 54A26C24
 P 1900 2500
-F 0 "#PWR040" H 1900 2500 30  0001 C CNN
+F 0 "#PWR041" H 1900 2500 30  0001 C CNN
 F 1 "GND" H 1900 2430 30  0001 C CNN
 F 2 "" H 1900 2500 60  0000 C CNN
@@
 	1900 4150 1900 4250
 $Comp
-L GND #PWR041
+L GND #PWR042
 U 1 1 54A272E7
 P 1900 4250
-F 0 "#PWR041" H 1900 4250 30  0001 C CNN
+F 0 "#PWR042" H 1900 4250 30  0001 C CNN
 F 1 "GND" H 1900 4180 30  0001 C CNN
 F 2 "" H 1900 4250 60  0000 C CNN
@@
 $EndComp
 $Comp
-L GND #PWR042
+L GND #PWR043
 U 1 1 54A63C22
 P 5950 4150
-F 0 "#PWR042" H 5950 4150 30  0001 C CNN
+F 0 "#PWR043" H 5950 4150 30  0001 C CNN
 F 1 "GND" H 5950 4080 30  0001 C CNN
 F 2 "" H 5950 4150 60  0000 C CNN
@@
 Connection ~ 7950 3750
 $Comp
-L GND #PWR043
+L GND #PWR044
 U 1 1 54A64006
 P 7950 4150
-F 0 "#PWR043" H 7950 4150 30  0001 C CNN
+F 0 "#PWR044" H 7950 4150 30  0001 C CNN
 F 1 "GND" H 7950 4080 30  0001 C CNN
 F 2 "" H 7950 4150 60  0000 C CNN
@@
 	3550 750  3550 800
 Wire Wire Line
-	3550 800  4500 800
-Wire Wire Line
 	3450 850  3450 1100
 Wire Wire Line
@@
 Wire Wire Line
 	3350 1300 4500 1300
-Connection ~ 3350 1300
 Wire Wire Line
 	4400 1550 4400 1750
@@
 $EndComp
 $Comp
-L GND #PWR044
+L GND #PWR045
 U 1 1 54ABE5DE
 P 5750 2250
-F 0 "#PWR044" H 5750 2250 30  0001 C CNN
+F 0 "#PWR045" H 5750 2250 30  0001 C CNN
 F 1 "GND" H 5750 2180 30  0001 C CNN
 F 2 "" H 5750 2250 60  0000 C CNN
@@
 $EndComp
 $Comp
-L GND #PWR045
+L GND #PWR046
 U 1 1 54ABE6E0
 P 8000 2250
-F 0 "#PWR045" H 8000 2250 30  0001 C CNN
+F 0 "#PWR046" H 8000 2250 30  0001 C CNN
 F 1 "GND" H 8000 2180 30  0001 C CNN
 F 2 "" H 8000 2250 60  0000 C CNN
@@
 Connection ~ 8000 1850
 Connection ~ 5750 1850
+$Comp
+L C C82
+U 1 1 54BBBF4C
+P 4000 800
+F 0 "C82" V 3950 900 40  0000 L CNN
+F 1 "0.1uF" V 4100 550 40  0000 L CNN
+F 2 "HERMESLITE:C_0805" H 4038 650 30  0001 C CNN
+F 3 "" H 4000 800 60  0000 C CNN
+	1    4000 800
+	0    1    1    0
+$EndComp
+Wire Wire Line
+	3550 800  3800 800
+Wire Wire Line
+	4200 800  4500 800
 $EndSCHEMATC

Commit message: BCD Filter update
Parts:
- removed P8: CONN_01X08, Pin_Headers:Pin_Header_Straight_1x08, symbol CONN_01X08
- removed U3, U4: TPIC6B595, Housings_SOIC:SOIC-20_7.5x12.8mm_Pitch1.27mm, symbol TPIC6B595
- added C83, C84, C85, C86, C87, C88: 0.01uF, HERMESLITE:C_0805, symbol C
- added K7: D3002, HERMESLITE:D3002, symbol D3002
- added Q4, Q5, Q6, Q7, Q8, Q9: 2N7000, SMD_Packages:SOT-23-GDS, symbol MOSFET_N
- added U1: 4028, SMD_Packages:TSSOP-16, symbol 4028
Connections:
- net +12V: now also K7.1 (+)
- net GND: now also C83.2, C84.2, C85.2, C86.2, C87.2, C88.2, Q4.2 (S), Q5.2 (S), Q6.2 (S), Q7.2 (S), Q8.2 (S), Q9.2 (S), U1.8 (VSS)
- net at C35.1, C37.1, L12.2: now also K7.4 (T1); no longer K6.7 (T2)
- net at C30.1, C35.2, L12.1: now also K7.7 (T2); no longer K6.9 (R2)
- net at K2.10 (-): now also C83.1, Q4.3 (D)
- net at K3.10 (-): now also C84.1, Q5.3 (D)
- net at K4.10 (-): now also C85.1, Q6.3 (D)
- net at K5.10 (-): now also C86.1, Q7.3 (D)
- net at K6.10 (-): now also C87.1, Q8.3 (D)
- net at C20.1, C24.2, L7.1: now also K6.7 (T2); no longer K6.2 (R1)
- new net: K6.2 (R1), K7.3 (C1)
- new net: K6.9 (R2), K7.8 (C2)
- new net: C88.1, K7.10 (-), Q9.3 (D)
- new net: K7.2 (R1), K7.9 (R2)
- new net: Q9.1 (G), U1.9 (S8)
- new net: Q8.1 (G), U1.4 (S7)
- new net: Q7.1 (G), U1.7 (S6)
- new net: Q6.1 (G), U1.6 (S5)
- new net: Q5.1 (G), U1.1 (S4)
- new net: Q4.1 (G), U1.15 (S3)
- new net #PTT: U1.10 (A)
- new net A: U1.11 (D)
- new net B: U1.12 (C)
- new net C: U1.13 (B)
- new net VDD: U1.16 (VDD)
- no-connect marks 8 -> 4
Other:
- note added: "#PTT is used to enable/disable TX. \nWhen #PTT is low, valid outputs\nexist on S1 thru S6. Otherwise the \nfilters are bypassed."
- note added: "Filter Settings for PowerSDR Hermes Ctrl\n(set for TX J16 Pins only)\n 1 2 3 4-7=Don't care\n160M 1 0 0\n80M 0 1 0\n60M 1 1 0\n40M 1 1 0\n30M 0 0 1\n20M 0 0 1\n17M 1 0 1\n15M 1 0 1\n12M 0 1 1\n10M 0 1 1"
- note added: "Note: There is a TX bypass present that is connected when no \nrelays are active. At this point, there is no bypass avail on RX. One could \nuse this bypass to deactivate TX LPFs if desired if there are sufficient LPFs \nin any attached external amps. You would place a value of 1 1 1 0 in the J16 \nTX assignment for all band positions."
- note removed: "10/12M\n17/15M\n30/20M\n60/40M\n80/75M\n160M\n/PTT"
- note removed: "For use with an external amplifier, such as the Hardrock 50, all of the filter\ncomponents and relays on this sheet can be omitted. Jumper pin 3 to pin 8\non K2 to bypass TXIN to TXOUT. U3 and U4 can be omitted if connector P8 is unused."
- moved on the sheet: C20, C24, C26, C30, C35, C37, L12, L7
