File: frontend/Megabasic/frontend.sch (KiCad schematic (older format))
At the start: 24 parts, among them CN1 EDGE, CN2 BREAKOUT, J1 SMA, J2 SMA, P6 CONN_01X12, Q1 2N7002, T1 4:1, T2 8:1, U1 4050, U2 74LS145

Commit message: first pass for Oshpark
Parts:
- removed CN2: BREAKOUT, HERMESLITE:BREAKOUT, symbol BREAKOUT
- removed J1, J2: SMA, HERMESLITE:SMA, symbol SMA
- added J1, J2: CONN_02X01, HERMESLITE:JUMPER, symbol CONN_02X01
- added P1, P2: CONN_01X02, Pin_Headers:Pin_Header_Straight_1x02, symbol CONN_01X02
- added P4: Control for Megaband, Pin_Headers:Pin_Header_Straight_1x07, symbol CONN_01X07
- added unit 5 of U1
- P3: renamed from P6; footprint Pin_Headers:Pin_Header_Straight_1x02 -> Pin_Headers:Pin_Header_Straight_1x12
- Q1: value 2N7002 -> FDV301
- R3: value 1.2K -> 4.99K
- R4: value 1.2K -> 4.99k
Connections:
- net GND: now also J1.1 (P1), J2.1 (P1), P4.1 (P1), P4.7 (P7), U1.8 (VSS)
- net VCC: now also U1.1 (VCC)
- net at CN1.A15 (3V): no longer CN1.A16 (3V)
- net at CN1.A17 (DGND): no longer CN1.A18 (DGND)
- net at CN1.B11 (PTT): now also U1.11; no longer Q1.G
- net at D1.2 (K), T2.2 (S2): now also J2.2 (P2), P2.1 (P1)
- net at T1.1 (S1): now also P1.2 (P2)
- net at T1.2 (S2): now also J1.2 (P2), P1.1 (P1)
- net at C4.1: now also P2.2 (P2)
- net at U1.2, U2.12 (P3): now also P4.3 (P3)
- net at U1.4, U2.13 (P2): now also P4.4 (P4)
- net at U1.6, U2.14 (P1): now also P4.5 (P5)
- net at U1.10, U2.15 (P0): now also P4.6 (P6)
- new net: P4.2 (P2), Q1.G, U1.12
- no-connect marks 2 -> 9
