File: frontend/basic superband pa/basic-superband-pa.sch (KiCad schematic (older format))
At the start: 70 parts, among them CN1 EDGE, K1 D3002, K2 D3002, P1 BNC, P2 CONN_02X01, Q3 RD16HHF1, T1 TRANSFO, T2 8:1, T3 4:1, T4 OUT_TRANSF, U1 LP2951-50D, U2 LVT827

Commit message: final 1.2 changes
Parts:
- added P3: Ext PTT, Pin_Headers:Pin_Header_Straight_1x02, symbol CONN_01X02
- added P4: 12-13.8v, Pin_Headers:Pin_Header_Straight_1x02, symbol CONN_01X02
- added R14: 4.99k, Resistors_SMD:R_0805_HandSoldering, symbol R
- C17, C28: value 0.1uF -> 1uF
- C22: value 10uF 16V -> 10uF 25V
- C23: value 220pF -> 270pF
- C7: value 47uF 16V -> 47uF 25V
- R1, R2: value 1.2k -> 270
- U2: value LVT827 -> LTV827
Connections:
- net GND: now also K2.2 (R1), P3.1 (P1), P4.1 (P1)
- net at C17.1, C26.2, C30.1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: now also P4.2 (P2), R14.2
- net at K2.3 (C1): now also P3.2 (P2)
- net at K2.4 (T1): now also R14.1
- no-connect marks 17 -> 14
Other:
- note added: "32 MHz Low Pass\n9 Turns #26 on T37-6 Toroid"
- note added: "Can Omit LEDs if desired"
- note added: "Ext PTT - active high, 12V"
- note added: "PTT - RX=low, TX=high\nUSEROUT4 = Band Select 0 = low,\nBand Select 1 = high"
- note removed: "Changed on 02-24 to a 32 MHz Low Pass\n9 Turns #26 on T37-6 Toroid"
- note removed: "PTT - RX=low, TX=high\nGPIO0 = BS0=low, BS1=high"
Changed lines of the file:
@@
 Sheet 1 1
 Title "Hermes-Lite Basic Superband 5W Power Amplifier"
-Date "10 March 2015"
-Rev "1.1"
+Date "19 March 2015"
+Rev "1.2"
 Comp "SofterHardware"
 Comment1 "AC9HY"
@@
 Text Notes 1400 7350 0    50   ~ 0
 BN-61-2402\n  2x4T #30
-Text Notes 1700 4400 0    60   ~ 0
-PTT - RX=low, TX=high\nGPIO0 = BS0=low, BS1=high
+Text Notes 1650 4500 0    60   ~ 0
+PTT - RX=low, TX=high\nUSEROUT4 = Band Select 0 = low,\nBand Select 1 =  high
 Text Notes 3600 6750 0    60   ~ 0
 (Band Specific Values)
@@
 P 5250 1750
 F 0 "C7" H 5300 1650 50  0000 L CNN
-F 1 "47uF 16V" H 5400 1750 50  0000 L CNN
+F 1 "47uF 25V" H 5400 1750 50  0000 L CNN
 F 2 "Capacitors_Tantalum_SMD:TantalC_SizeD_EIA-7343_HandSoldering" H 5250 1750 60  0001 C CNN
 F 3 "" H 5250 1750 60  0000 C CNN
@@
 P 6350 2550
 F 0 "C17" H 6350 2650 40  0000 L CNN
-F 1 "0.1uF" H 6150 2650 40  0000 L CNN
+F 1 "1uF" H 6150 2650 40  0000 L CNN
 F 2 "HERMESLITE:C_0805" H 6388 2400 30  0001 C CNN
 F 3 "" H 6350 2550 60  0000 C CNN
@@
 P 9200 3100
 F 0 "C22" V 9250 2900 50  0000 L CNN
-F 1 "10uF 16V" V 9050 2900 50  0000 L CNN
+F 1 "10uF 25V" V 9050 2900 50  0000 L CNN
 F 2 "Capacitors_Tantalum_SMD:TantalC_SizeC_EIA-6032_HandSoldering" H 9200 3100 60  0001 C CNN
 F 3 "" H 9200 3100 60  0000 C CNN
@@
 P 9200 4500
 F 0 "C23" H 9250 4600 40  0000 L CNN
-F 1 "220pF" H 9000 4600 40  0000 L CNN
+F 1 "270pF" H 9000 4600 40  0000 L CNN
 F 2 "HERMESLITE:C_0805" H 9238 4350 30  0001 C CNN
 F 3 "" H 9200 4500 60  0000 C CNN
@@
 	1    0    0    -1
 $EndComp
-NoConn ~ 3650 5600
-NoConn ~ 4450 5500
-NoConn ~ 4450 5700
 $Comp
 L GND #PWR024
@@
 P 6550 3200
 F 0 "C28" H 6650 3300 40  0000 L CNN
-F 1 "0.1uF" H 6550 3100 40  0000 L CNN
+F 1 "1uF" H 6550 3100 40  0000 L CNN
 F 2 "HERMESLITE:C_0805" H 6588 3050 30  0001 C CNN
 F 3 "" H 6550 3200 60  0000 C CNN
@@
 P 3050 4700
 F 0 "U2" H 2860 4890 40  0000 C CNN
-F 1 "LVT827" H 3210 4510 40  0000 C CNN
+F 1 "LTV827" H 3210 4510 40  0000 C CNN
 F 2 "Power_Integrations:SMD-8" H 2850 4520 30  0001 C CIN
 F 3 "" H 3050 4700 60  0000 C CNN
@@
 P 2450 4800
 F 0 "R1" V 2530 4800 40  0000 C CNN
-F 1 "1.2k" V 2457 4801 40  0000 C CNN
+F 1 "270" V 2457 4801 40  0000 C CNN
 F 2 "Resistors_SMD:R_0805_HandSoldering" V 2380 4800 30  0001 C CNN
 F 3 "" H 2450 4800 30  0000 C CNN
@@
 P 2450 5750
 F 0 "U2" H 2260 5940 40  0000 C CNN
-F 1 "LVT827" H 2610 5560 40  0000 C CNN
-F 2 "Power_Integrations:SMD-8" H 2250 5570 30  0000 C CIN
+F 1 "LTV827" H 2610 5560 40  0000 C CNN
+F 2 "Power_Integrations:SMD-8" H 2250 5570 30  0001 C CIN
 F 3 "" H 2450 5750 60  0000 C CNN
 	2    2450 5750
@@
 P 1850 5850
 F 0 "R2" V 1930 5850 40  0000 C CNN
-F 1 "1.2k" V 1857 5851 40  0000 C CNN
+F 1 "270" V 1857 5851 40  0000 C CNN
 F 2 "Resistors_SMD:R_0805_HandSoldering" V 1780 5850 30  0001 C CNN
 F 3 "" H 1850 5850 30  0000 C CNN
@@
 	7050 900  7200 900
 Text Notes 8500 4100 0    50   ~ 0
-Changed on 02-24 to a 32 MHz Low Pass\n9 Turns #26 on T37-6 Toroid
+32 MHz Low Pass\n9 Turns #26 on T37-6 Toroid
 $Comp
 L C C1
@@
 	9400 2100 9600 2100
 Connection ~ 9600 2350
+$Comp
+L CONN_01X02 P3
+U 1 1 550BDA20
+P 1700 5050
+F 0 "P3" H 1700 5200 50  0000 C CNN
+F 1 "Ext PTT" V 1800 5050 50  0000 C CNN
+F 2 "Pin_Headers:Pin_Header_Straight_1x02" H 1700 5050 60  0001 C CNN
+F 3 "" H 1700 5050 60  0000 C CNN
+	1    1700 5050
+	-1   0    0    1
+$EndComp
+Wire Wire Line
+	1900 5100 2000 5100
+Wire Wire Line
+	2000 5100 2000 5200
+$Comp
+L GND #PWR037
+U 1 1 550BDD15
+P 2000 5200
+F 0 "#PWR037" H 2000 5200 30  0001 C CNN
+F 1 "GND" H 2000 5130 30  0001 C CNN
+F 2 "" H 2000 5200 60  0000 C CNN
+F 3 "" H 2000 5200 60  0000 C CNN
+	1    2000 5200
+	1    0    0    -1
+$EndComp
+Wire Wire Line
+	1900 5000 2050 5000
+Wire Wire Line
+	2050 5000 2050 5100
+Wire Wire Line
+	2050 5100 2650 5100
+Wire Wire Line
+	2650 5100 2650 5300
+Wire Wire Line
+	2650 5300 3500 5300
+Wire Wire Line
+	3500 5300 3500 5600
+Wire Wire Line
+	3500 5600 3650 5600
+Wire Wire Line
+	4450 5700 4800 5700
+Wire Wire Line
+	4800 5700 4800 5900
+$Comp
+L GND #PWR038
+U 1 1 550BE0EF
+P 4800 5900
+F 0 "#PWR038" H 4800 5900 30  0001 C CNN
+F 1 "GND" H 4800 5830 30  0001 C CNN
+F 2 "" H 4800 5900 60  0000 C CNN
+F 3 "" H 4800 5900 60  0000 C CNN
+	1    4800 5900
+	1    0    0    -1
+$EndComp
+Wire Wire Line
+	3550 5000 3550 5400
+Connection ~ 3550 5400
+$Comp
+L R R14
+U 1 1 550BE620
+P 4800 5250
+F 0 "R14" V 4880 5250 40  0000 C CNN
+F 1 "4.99k" V 4807 5251 40  0000 C CNN
+F 2 "Resistors_SMD:R_0805_HandSoldering" V 4730 5250 30  0001 C CNN
+F 3 "" H 4800 5250 30  0000 C CNN
+	1    4800 5250
+	-1   0    0    1
+$EndComp
+Wire Wire Line
+	3550 5000 4800 5000
+Wire Wire Line
+	4800 5500 4450 5500
+$Comp
+L CONN_01X02 P4
+U 1 1 550EC103
+P 8600 950
+F 0 "P4" H 8600 1100 50  0000 C CNN
+F 1 "12-13.8v" V 8700 950 50  0000 C CNN
+F 2 "Pin_Headers:Pin_Header_Straight_1x02" H 8600 950 60  0001 C CNN
+F 3 "" H 8600 950 60  0000 C CNN
+	1    8600 950
+	0    -1   -1   0
+$EndComp
+$Comp
+L GND #PWR039
+U 1 1 550ED567
+P 8550 1150
+F 0 "#PWR039" H 8550 1150 30  0001 C CNN
+F 1 "GND" H 8550 1080 30  0001 C CNN
+F 2 "" H 8550 1150 60  0000 C CNN
+F 3 "" H 8550 1150 60  0000 C CNN
+	1    8550 1150
+	1    0    0    -1
+$EndComp
+Wire Wire Line
+	8650 1150 8650 1550
+Connection ~ 8650 1550
+Text Notes 5500 1250 0    50   ~ 0
+Can Omit LEDs if desired
+Text Notes 1500 5350 0    50   ~ 0
+Ext PTT - active high, 12V
 $EndSCHEMATC

Commit message: cleanup, minor superband changes
Parts:
- removed C18, C24: 150pF, HERMESLITE:C_0805, symbol C
- removed C23: 270pF, HERMESLITE:C_0805, symbol C
- removed L11, L9: 240nH, Choke_Toroid_ThroughHole:Choke_Toroid_6,5x13mm_Vertical, symbol INDUCTOR_SMALL
- removed P2: CONN_02X01, Pin_Headers:Pin_Header_Straight_2x01, symbol CONN_02X01
- removed T1: TRANSFO, Socket_Strips:Socket_Strip_Straight_2x02, symbol TRANSFO
- removed U2: LTV827, Power_Integrations:SMD-8, symbol PC827
- added D4: DIODESCH2, HERMESLITE:SOD323, symbol DIODESCH2
- added Q1, Q2: FDV301, HERMESLITE:SOT-23-GDS, symbol MOSFET_N
- added R15, R16: 10k, Resistors_SMD:R_0805_HandSoldering, symbol R
- R1, R2: value 270 -> 499
- R10, R12: value DNI -> 270
- R11: value 0 -> 18
Connections:
- net /PTT: now also Q1.3 (D)
- net BAND1: now also Q2.3 (D)
- net GND: now also P1.2 (Ext), D4.2 (K), Q1.2 (S), Q2.2 (S), R15.1, R16.1; no longer R1.2, R2.2
- net PTT: now also R1.2
- net USEROUT4: now also R2.2
- net at K2.9 (R2), T2.1 (S1): now also D4.1 (A)
- net at P1.1 (In): now also K1.8 (C2)
- net at T4.4 (SA): now also C29.2
- net at R1.1: now also Q1.1 (G), R16.2
- net at R2.1: now also Q2.1 (G), R15.2
Other:
- note added: "3db Attenuator"
- note removed: "BN-61-2402\n 2x4T #30"
- note removed: "Ground\nOption"
- moved on the sheet: P3
